Commit message: update for inmoov urdf. now all joints have correct orientation except for right wrist and right shoulder

File: inmoov_description/robots/inmoov.urdf (robot description, URDF)
Before this commit: robot inmoov, 86 links, 85 joints
Links:
- added link head_tilt; visual mesh filename=package://inmoov_description/meshes/virtual.stl scale=0.001 0.001 0.001
Joints:
- removed joint left_index2
- removed joint left_middle2
- removed joint left_pinky2
- removed joint left_ring2
- removed joint left_thumb2
- removed joint right_eye_leftright
- removed joint right_index2
- removed joint right_middle2
- removed joint right_pinky2
- removed joint right_ring2
- removed joint right_thumb2
- added joint eye_leftright: type revolute, parent eyesupport, child right_eyesupport, origin xyz=0.033 0 -0.0036 rpy=0 0 0, axis 0 0 1, limit lower=-0.45 upper=0.45 effort=1000.0 velocity=0.5
- added joint head_tilt: type revolute, parent torso, child head_tilt, origin xyz=-0.001 -0.0315 0.4551 rpy=0 0 0, axis 0 1 0, limit lower=-0.30 upper=0.30 effort=1000.0 velocity=0.5
- added joint left_index: type revolute, parent left_index1, child left_index2, origin xyz=0 0.001 -0.03595 rpy=0 0 0, axis 1 0 0, limit lower=0 upper=1.5 effort=1000.0 velocity=0.5
- added joint left_middle: type revolute, parent left_middle1, child left_middle2, origin xyz=0 0.000 -0.0389 rpy=0 0 0, axis 1 0 0, limit lower=0 upper=1.5 effort=1000.0 velocity=0.5
- added joint left_pinky: type revolute, parent left_pinky1, child left_pinky2, origin xyz=0.046 -0 -0.0228 rpy=0 -0.93 0, axis 1 0 0, limit lower=0 upper=1.5 effort=1000.0 velocity=0.5
- added joint left_ring: type revolute, parent left_ring1, child left_ring2, origin xyz=0.0351 0.00126 -0.0166 rpy=0 -0.7775 0, axis 1 0 0, limit lower=0 upper=1.5 effort=1000.0 velocity=0.5
- added joint left_thumb: type revolute, parent left_thumb1, child left_thumb2, origin xyz=0.02725 -0.0006 0.014 rpy=0 -2.3 0.3, axis 1 0 0, limit lower=0 upper=1.5 effort=1000.0 velocity=0.5
- added joint right_index: type revolute, parent right_index1, child right_index2, origin xyz=0 0.001 -0.03595 rpy=0 0 0, axis 1 0 0, limit lower=0 upper=1.5 effort=1000.0 velocity=0.5
- added joint right_middle: type revolute, parent right_middle1, child right_middle2, origin xyz=0 0.000 -0.0389 rpy=0 0 0, axis 1 0 0, limit lower=0 upper=1.5 effort=1000.0 velocity=0.5
- added joint right_pinky: type revolute, parent right_pinky1, child right_pinky2, origin xyz=-0.046 -0 -0.0228 rpy=0 0.93 0, axis 1 0 0, limit lower=0 upper=1.5 effort=1000.0 velocity=0.5
- added joint right_ring: type revolute, parent right_ring1, child right_ring2, origin xyz=-0.0351 0.00126 -0.0166 rpy=0 0.7775 0, axis 1 0 0, limit lower=0 upper=1.5 effort=1000.0 velocity=0.5
- added joint right_thumb: type revolute, parent right_thumb1, child right_thumb2, origin xyz=-0.02725 -0.0006 0.014 rpy=0 2.3 -0.3, axis 1 0 0, limit lower=0 upper=1.5 effort=1000.0 velocity=0.5
- joint head_updown: origin xyz=-0.001 -0.0315 0.4551 rpy=0 0 0 -> xyz=0 0 0 rpy=0 0 0; parent torso -> head_tilt
- joint jaw: limit lower=0 upper=-0.15 effort=1000.0 velocity=0.5 -> lower=0 upper=0.15 effort=1000.0 velocity=0.5; origin xyz=-0.001 0.0375 0.0437 rpy=-0.085 0 0 -> xyz=-0.001 0.0375 0.0437 rpy=0.085 0 3.1415
- joint left_bicep: limit lower=0.75 upper=1.57 effort=1000.0 velocity=0.5 -> lower=0.4 upper=1.57 effort=1000.0 velocity=0.5
- joint left_cover_handpinky: origin xyz=-0.0205 0.01 -0.0069 rpy=0 0.7 0 -> xyz=0.0205 -0.01 -0.0069 rpy=0 -0.7 0
- joint left_cover_handring: origin xyz=-0.015 0.009 -0.0008 rpy=0 0.7 0 -> xyz=0.015 -0.009 -0.0008 rpy=0 -0.7 0
- joint left_cover_index: origin xyz=0 0.0071 -0.012 rpy=0.05 0 0 -> xyz=0 -0.0071 -0.012 rpy=-0.05 0 0
- joint left_cover_middle: origin xyz=0 0.0071 -0.012 rpy=0.05 0 0 -> xyz=0 -0.0071 -0.012 rpy=0.05 0 0
- joint left_cover_pinky: origin xyz=0 0.0071 -0.0105 rpy=0.05 -0.1 0 -> xyz=0 -0.005 -0.0105 rpy=0.05 0.1 0
- joint left_cover_ring: origin xyz=0 0.0071 -0.011 rpy=0.05 -0.1 0 -> xyz=0 -0.005 -0.011 rpy=0.05 0.1 0
- joint left_cover_thumb: origin xyz=0.02125 0.01 0.0047 rpy=0 -3.2 0 -> xyz=0.02125 -0.01 -0.0047 rpy=0 -3.1 0
- joint left_eye_leftright: mimic (none) -> joint=eye_leftright multiplier=1 offset=0
- joint left_index1: limit lower=-1.57 upper=0 effort=1000.0 velocity=0.5 -> lower=0 upper=1.5 effort=1000.0 velocity=0.5; mimic (none) -> joint=left_index multiplier=1 offset=0; origin xyz=0.0342 -0.0015 -0.119 rpy=0 -0.1 0 -> xyz=0.0342 -0.0015 -0.119 rpy=0 0.1 3.1415
- joint left_index3: limit lower=-1.57 upper=0 effort=1000.0 velocity=0.5 -> lower=0 upper=1.5 effort=1000.0 velocity=0.5; mimic (none) -> joint=left_index multiplier=1 offset=0
- joint left_middle1: limit lower=-1.57 upper=0 effort=1000.0 velocity=0.5 -> lower=0 upper=1.5 effort=1000.0 velocity=0.5; mimic (none) -> joint=left_middle multiplier=1 offset=0; origin xyz=0.007 -0.00175 -0.12325 rpy=0 0 0 -> xyz=0.007 -0.00175 -0.12325 rpy=0 0 3.1415
- joint left_middle3: mimic (none) -> joint=left_middle multiplier=1 offset=0
- joint left_pinky1: mimic (none) -> joint=left_pinky multiplier=0.1 offset=0; origin xyz=-0.027 0 -0.0555 rpy=0 -0.7 0 -> xyz=-0.027 0 -0.0555 rpy=0 0.7 3.1415
- joint left_pinky3: mimic (none) -> joint=left_pinky multiplier=1 offset=0
- joint left_pinky4: mimic (none) -> joint=left_pinky multiplier=1 offset=0
- joint left_ring1: mimic (none) -> joint=left_ring multiplier=0.1 offset=0; origin xyz=-0.00705 0 -0.0794 rpy=0 -0.7 0 -> xyz=-0.00705 0 -0.0794 rpy=0 0.7 3.1415
- joint left_ring3: mimic (none) -> joint=left_ring multiplier=1 offset=0
- joint left_ring4: mimic (none) -> joint=left_ring multiplier=1 offset=0
- joint left_shoulder_up: origin xyz=0.012 0 -0.04 rpy=0 0 0 -> xyz=-0.012 0 -0.04 rpy=0 0 0
- joint left_thumb1: mimic (none) -> joint=left_thumb multiplier=0.75 offset=0; origin xyz=0.029 0 -0.0577 rpy=0 -0.1 0 -> xyz=0.029 0 -0.0577 rpy=3.1415 -0.1 0
- joint left_thumb3: mimic (none) -> joint=left_thumb multiplier=1 offset=0
- joint right_bicep: limit lower=0.75 upper=1.57 effort=1000.0 velocity=0.5 -> lower=0.4 upper=1.57 effort=1000.0 velocity=0.5
- joint right_cover_handpinky: origin xyz=0.0205 0.01 -0.0069 rpy=0 -0.7 0 -> xyz=-0.0205 -0.01 -0.0069 rpy=0 0.7 0
- joint right_cover_handring: origin xyz=0.015 0.009 -0.0008 rpy=0 -0.7 0 -> xyz=-0.015 -0.009 -0.0008 rpy=0 0.7 0
- joint right_cover_index: origin xyz=0 0.0071 -0.012 rpy=-0.05 0 0 -> xyz=0 -0.0071 -0.012 rpy=0.05 0 0
- joint right_cover_middle: origin xyz=0 0.0071 -0.012 rpy=-0.05 0 0 -> xyz=0 -0.0071 -0.012 rpy=-0.05 0 0
- joint right_cover_pinky: origin xyz=0 0.0071 -0.0105 rpy=-0.05 0.1 0 -> xyz=0 -0.005 -0.0105 rpy=-0.05 -0.1 0
- joint right_cover_ring: origin xyz=0 0.0071 -0.011 rpy=-0.05 0.1 0 -> xyz=0 -0.005 -0.011 rpy=-0.05 -0.1 0
- joint right_cover_thumb: origin xyz=-0.02125 0.01 0.0047 rpy=0 3.2 0 -> xyz=-0.02125 -0.01 -0.0047 rpy=0 3.1 0
- joint right_index1: limit lower=-1.57 upper=0 effort=1000.0 velocity=0.5 -> lower=0 upper=1.5 effort=1000.0 velocity=0.5; mimic (none) -> joint=right_index multiplier=1 offset=0; origin xyz=-0.0342 -0.0015 -0.119 rpy=0 0.1 0 -> xyz=-0.0342 -0.0015 -0.119 rpy=0 -0.1 3.1415
- joint right_index3: limit lower=-1.57 upper=0 effort=1000.0 velocity=0.5 -> lower=0 upper=1.5 effort=1000.0 velocity=0.5; mimic (none) -> joint=right_index multiplier=1 offset=0
- joint right_middle1: limit lower=-1.57 upper=0 effort=1000.0 velocity=0.5 -> lower=0 upper=1.5 effort=1000.0 velocity=0.5; mimic (none) -> joint=right_middle multiplier=1 offset=0; origin xyz=-0.007 -0.00175 -0.12325 rpy=0 0 0 -> xyz=-0.007 -0.00175 -0.12325 rpy=0 0 3.1415
- joint right_middle3: mimic (none) -> joint=right_middle multiplier=1 offset=0
- joint right_pinky1: mimic (none) -> joint=right_pinky multiplier=-0.1 offset=0; origin xyz=0.027 0 -0.0555 rpy=0 0.7 0 -> xyz=0.027 0 -0.0555 rpy=0 -0.7 3.1415
- joint right_pinky3: mimic (none) -> joint=right_pinky multiplier=1 offset=0
- joint right_pinky4: mimic (none) -> joint=right_pinky multiplier=1 offset=0
- joint right_ring1: mimic (none) -> joint=right_ring multiplier=-0.1 offset=0; origin xyz=0.00705 0 -0.0794 rpy=0 0.7 0 -> xyz=0.00705 0 -0.0794 rpy=0 -0.7 3.1415
- joint right_ring3: mimic (none) -> joint=right_ring multiplier=1 offset=0
- joint right_ring4: mimic (none) -> joint=right_ring multiplier=1 offset=0
- joint right_shoulder_side: limit lower=0 upper=-0.75 effort=1000.0 velocity=0.5 -> lower=-0.75 upper=0 effort=1000.0 velocity=0.5
- joint right_shoulder_up: origin xyz=-0.012 0 -0.04 rpy=0 0 0 -> xyz=0.012 0 -0.04 rpy=0 0 0
- joint right_thumb1: mimic (none) -> joint=right_thumb multiplier=-0.75 offset=0; origin xyz=-0.029 0 -0.0577 rpy=0 0.1 0 -> xyz=-0.029 0 -0.0577 rpy=3.1415 0.1 0
- joint right_thumb3: mimic (none) -> joint=right_thumb multiplier=1 offset=0

File: inmoov_description/robots/inmoov.urdf.xacro (robot description, xacro)
@@ -31,4 +31,13 @@
     </visual>
   </link>
+  <link name="head_tilt">
+    <visual>
+      <geometry>
+        <mesh filename="package://inmoov_description/meshes/virtual.stl" scale="0.001 0.001 0.001"/>
+      </geometry>
+      <origin rpy="0 0 0" xyz="0 0 0"/>
+      <xacro:frame_color/>
+    </visual>
+  </link>
   <joint name="pedestal_to_mid_stomach" type="fixed">
     <parent link="pedestal"/>
@@ -37,9 +46,16 @@
   </joint>
   <xacro:torso side="right" covers="yes" />
+  <joint name="head_tilt" type="revolute">
+   <axis xyz="0 1 0"/>
+   <limit effort="1000.0" lower="-0.30" upper="0.30" velocity="0.5"/>
+   <origin rpy="0 0 0" xyz="-0.001 -0.0315 0.4551"/>
+   <parent link="torso"/>
+   <child link="head_tilt"/>
+  </joint>
   <joint name="head_updown" type="revolute">
    <axis xyz="1 0 0"/>
    <limit effort="1000.0" lower="-0.30" upper="0.30" velocity="0.5"/>
-   <origin rpy="0 0 0" xyz="-0.001 -0.0315 0.4551"/>
-   <parent link="torso"/>
+   <origin rpy="0 0 0" xyz="0 0 0"/>
+   <parent link="head_tilt"/>
    <child link="head_base"/>
   </joint>
@@ -54,5 +70,5 @@
   <joint name="right_shoulder_side" type="revolute">
    <axis xyz="0 1 0"/>
-   <limit effort="1000.0" lower="0" upper="-0.75" velocity="0.5"/>
+   <limit effort="1000.0" lower="-0.75" upper="0" velocity="0.5"/>
    <origin rpy="0 0 0" xyz="0.143 0 0.298"/>
    <parent link="torso"/>

File: inmoov_description/robots/inmoov_head.urdf (robot description, URDF)
Before this commit: robot inmoov_hand, 17 links, 16 joints
Joints:
- removed joint right_eye_leftright
- added joint eye_leftright: type revolute, parent eyesupport, child right_eyesupport, origin xyz=0.033 0 -0.0036 rpy=0 0 0, axis 0 0 1, limit lower=-0.45 upper=0.45 effort=1000.0 velocity=0.5
- joint eyes_updown: limit lower=-1.57 upper=1.57 effort=1000.0 velocity=0.5 -> lower=-0.45 upper=0.45 effort=1000.0 velocity=0.5
- joint jaw: limit lower=0 upper=-0.15 effort=1000.0 velocity=0.5 -> lower=0 upper=0.15 effort=1000.0 velocity=0.5; origin xyz=-0.001 0.0375 0.0437 rpy=-0.085 0 0 -> xyz=-0.001 0.0375 0.0437 rpy=0.085 0 3.1415
- joint left_ear: origin xyz=-0.059 0.035 0.0437 rpy=0 0 0 -> xyz=-0.056 0.035 0.0437 rpy=0 0 0
- joint left_eye_leftright: limit lower=-1.57 upper=1.57 effort=1000.0 velocity=0.5 -> lower=-0.45 upper=0.45 effort=1000.0 velocity=0.5; mimic (none) -> joint=eye_leftright multiplier=1 offset=0
- joint right_ear: origin xyz=0.059 0.035 0.0437 rpy=0 0 0 -> xyz=0.056 0.035 0.0437 rpy=0 0 0

File: inmoov_description/robots/inmoov_right_hand.urdf (robot description, URDF)
Before this commit: robot inmoov_hand, 27 links, 26 joints
Joints:
- removed joint right_index2
- removed joint right_middle2
- removed joint right_pinky2
- removed joint right_ring2
- removed joint right_thumb2
- added joint right_index: type revolute, parent right_index1, child right_index2, origin xyz=0 0.001 -0.03595 rpy=0 0 0, axis 1 0 0, limit lower=0 upper=1.5 effort=1000.0 velocity=0.5
- added joint right_middle: type revolute, parent right_middle1, child right_middle2, origin xyz=0 0.000 -0.0389 rpy=0 0 0, axis 1 0 0, limit lower=0 upper=1.5 effort=1000.0 velocity=0.5
- added joint right_pinky: type revolute, parent right_pinky1, child right_pinky2, origin xyz=-0.046 -0 -0.0228 rpy=0 0.93 0, axis 1 0 0, limit lower=0 upper=1.5 effort=1000.0 velocity=0.5
- added joint right_ring: type revolute, parent right_ring1, child right_ring2, origin xyz=-0.0351 0.00126 -0.0166 rpy=0 0.7775 0, axis 1 0 0, limit lower=0 upper=1.5 effort=1000.0 velocity=0.5
- added joint right_thumb: type revolute, parent right_thumb1, child right_thumb2, origin xyz=-0.02725 -0.0006 0.014 rpy=0 2.3 -0.3, axis 1 0 0, limit lower=0 upper=1.5 effort=1000.0 velocity=0.5
- joint right_cover_handpinky: origin xyz=0.0205 0.01 -0.0069 rpy=0 -0.7 0 -> xyz=-0.0205 -0.01 -0.0069 rpy=0 0.7 0
- joint right_cover_handring: origin xyz=0.015 0.009 -0.0008 rpy=0 -0.7 0 -> xyz=-0.015 -0.009 -0.0008 rpy=0 0.7 0
- joint right_cover_index: origin xyz=0 0.0071 -0.012 rpy=-0.05 0 0 -> xyz=0 -0.0071 -0.012 rpy=0.05 0 0
- joint right_cover_middle: origin xyz=0 0.0071 -0.012 rpy=-0.05 0 0 -> xyz=0 -0.0071 -0.012 rpy=-0.05 0 0
- joint right_cover_pinky: origin xyz=0 0.0071 -0.0105 rpy=-0.05 0.1 0 -> xyz=0 -0.005 -0.0105 rpy=-0.05 -0.1 0
- joint right_cover_ring: origin xyz=0 0.0071 -0.011 rpy=-0.05 0.1 0 -> xyz=0 -0.005 -0.011 rpy=-0.05 -0.1 0
- joint right_cover_thumb: origin xyz=-0.02125 0.01 0.0047 rpy=0 3.2 0 -> xyz=-0.02125 -0.01 -0.0047 rpy=0 3.1 0
- joint right_index1: limit lower=-1.57 upper=0 effort=1000.0 velocity=0.5 -> lower=0 upper=1.5 effort=1000.0 velocity=0.5; mimic (none) -> joint=right_index multiplier=1 offset=0; origin xyz=-0.0342 -0.0015 -0.119 rpy=0 0.1 0 -> xyz=-0.0342 -0.0015 -0.119 rpy=0 -0.1 3.1415
- joint right_index3: limit lower=-1.57 upper=0 effort=1000.0 velocity=0.5 -> lower=0 upper=1.5 effort=1000.0 velocity=0.5; mimic (none) -> joint=right_index multiplier=1 offset=0
- joint right_middle1: limit lower=-1.57 upper=0 effort=1000.0 velocity=0.5 -> lower=0 upper=1.5 effort=1000.0 velocity=0.5; mimic (none) -> joint=right_middle multiplier=1 offset=0; origin xyz=-0.007 -0.00175 -0.12325 rpy=0 0 0 -> xyz=-0.007 -0.00175 -0.12325 rpy=0 0 3.1415
- joint right_middle3: mimic (none) -> joint=right_middle multiplier=1 offset=0
- joint right_pinky1: mimic (none) -> joint=right_pinky multiplier=0.1 offset=0; origin xyz=0.0270 0 -0.0555 rpy=0 0.7 0 -> xyz=0.027 0 -0.0555 rpy=0 -0.7 3.1415
- joint right_pinky3: mimic (none) -> joint=right_pinky multiplier=1 offset=0
- joint right_pinky4: mimic (none) -> joint=right_pinky multiplier=1 offset=0
- joint right_ring1: mimic (none) -> joint=right_ring multiplier=0.1 offset=0; origin xyz=0.00705 0 -0.0794 rpy=0 0.7 0 -> xyz=0.00705 0 -0.0794 rpy=0 -0.7 3.1415
- joint right_ring3: mimic (none) -> joint=right_ring multiplier=1 offset=0
- joint right_ring4: mimic (none) -> joint=right_ring multiplier=1 offset=0
- joint right_thumb1: mimic (none) -> joint=right_thumb multiplier=-0.75 offset=0; origin xyz=-0.029 0 -0.0577 rpy=0 0.1 0 -> xyz=-0.029 0 -0.0577 rpy=3.1415 0.1 0
- joint right_thumb3: mimic (none) -> joint=right_thumb multiplier=1 offset=0

File: inmoov_description/robots/inmoov_right_hand.urdf.xacro (robot description, xacro)
@@ -14,5 +14,5 @@
     </visual>
   </link>
-<xacro:hand side="right" flip="0" covers="yes" />
+  <xacro:hand side="right" neg="1" flip="0" covers="yes" />
   <joint name="base_to_hand" type="revolute">
    <axis xyz="0 0 1"/>

File: inmoov_description/urdf/asmArm.urdf.xacro (robot description, xacro)
@@ -51,5 +51,5 @@
     <axis xyz="1 0 0"/>
     <limit effort="1000.0" lower="0" upper="3.14" velocity="0.5"/>
-    <origin rpy="0 0 0" xyz="${flip * -0.012} 0 -0.04"/>
+    <origin rpy="0 0 0" xyz="${flip * 0.012} 0 -0.04"/>
     <parent link="${side}_shoulder_base"/>
     <child link="${side}_shoulder"/>
@@ -64,5 +64,5 @@
   <joint name="${side}_bicep" type="revolute">
     <axis xyz="1 0 0"/>
-    <limit effort="1000.0" lower="0.75" upper="1.57" velocity="0.5"/>
+    <limit effort="1000.0" lower="0.4" upper="1.57" velocity="0.5"/>
     <origin rpy="0 0 0" xyz="0 -0.0278 -0.2235"/>
     <parent link="${side}_bicep"/>

File: inmoov_description/urdf/asmFace.urdf.xacro (robot description, xacro)
@@ -29,5 +29,5 @@
   </link>
 <xacro:asmEye side="right" flip="1" />
-  <joint name="right_eye_leftright" type="revolute">
+  <joint name="eye_leftright" type="revolute">
    <axis xyz="0 0 1"/>
    <limit effort="1000.0" lower="-0.45" upper="0.45" velocity="0.5"/>
@@ -40,4 +40,5 @@
    <axis xyz="0 0 1"/>
    <limit effort="1000.0" lower="-0.45" upper="0.45" velocity="0.5"/>
+   <mimic joint="eye_leftright" multiplier="1" offset="0"/>
    <origin rpy="0 0 0" xyz="-0.033 0 -0.0036"/>
    <parent link="eyesupport"/>
