Commit message: update for inmoov urdf. now all joints have correct orientation except for right wrist and right shoulder

File: inmoov_description/urdf/asmHand.urdf.xacro (robot description, xacro)
@@ -17,5 +17,5 @@
         <mesh filename="package://inmoov_description/meshes/${side}_thumb5_1.stl" scale="0.001 0.001 0.001"/>
       </geometry>
-      <origin rpy="0 0 0" xyz="0 0 0"/>
+      <origin rpy="3.1415 0 0" xyz="0 0 0"/>
       <xacro:frame_color/>
     </visual>
@@ -26,5 +26,5 @@
         <mesh filename="package://inmoov_description/meshes/thumb5_2.stl" scale="0.001 0.001 0.001"/>
       </geometry>
-      <origin rpy="0 0 0" xyz="0 0 0"/>
+      <origin rpy="0 0 3.1415" xyz="0 0 0"/>
       <xacro:frame_color/>
     </visual>
@@ -35,5 +35,5 @@
         <mesh filename="package://inmoov_description/meshes/thumb5_3.stl" scale="0.001 0.001 0.001"/>
       </geometry>
-      <origin rpy="0 0 0" xyz="0 0 0"/>
+      <origin rpy="0 0 3.1415" xyz="0 0 0"/>
       <xacro:frame_color/>
     </visual>
@@ -44,5 +44,5 @@
         <mesh filename="package://inmoov_description/meshes/index3_1.stl" scale="0.001 0.001 0.001"/>
       </geometry>
-      <origin rpy="0 0 0" xyz="0 0 0"/>
+      <origin rpy="0 0 3.1415" xyz="0 0 0"/>
       <xacro:frame_color/>
     </visual>
@@ -53,5 +53,5 @@
         <mesh filename="package://inmoov_description/meshes/index3_2.stl" scale="0.001 0.001 0.001"/>
       </geometry>
-      <origin rpy="0 0 0" xyz="0 0 0"/>
+      <origin rpy="0 0 3.1415" xyz="0 0 0"/>
       <xacro:frame_color/>
     </visual>
@@ -62,5 +62,5 @@
         <mesh filename="package://inmoov_description/meshes/index3_3.stl" scale="0.001 0.001 0.001"/>
       </geometry>
-      <origin rpy="0 0 0" xyz="0 0 0"/>
+      <origin rpy="0 0 3.1415" xyz="0 0 0"/>
       <xacro:frame_color/>
     </visual>
@@ -71,5 +71,5 @@
         <mesh filename="package://inmoov_description/meshes/middle3_1.stl" scale="0.001 0.001 0.001"/>
       </geometry>
-      <origin rpy="0 0 0" xyz="0 0 0"/>
+      <origin rpy="0 0 3.1415" xyz="0 0 0"/>
       <xacro:frame_color/>
     </visual>
@@ -80,5 +80,5 @@
         <mesh filename="package://inmoov_description/meshes/middle3_2.stl" scale="0.001 0.001 0.001"/>
       </geometry>
-      <origin rpy="0 0 0" xyz="0 0 0"/>
+      <origin rpy="0 0 3.1415" xyz="0 0 0"/>
       <xacro:frame_color/>
     </visual>
@@ -89,5 +89,5 @@
         <mesh filename="package://inmoov_description/meshes/middle3_3.stl" scale="0.001 0.001 0.001"/>
       </geometry>
-      <origin rpy="0 0 0" xyz="0 0 0"/>
+      <origin rpy="0 0 3.1415" xyz="0 0 0"/>
       <xacro:frame_color/>
     </visual>
@@ -98,5 +98,5 @@
         <mesh filename="package://inmoov_description/meshes/${side}_ring3_1.stl" scale="0.001 0.001 0.001"/>
       </geometry>
-      <origin rpy="0 0 0" xyz="0 0 0"/>
+      <origin rpy="0 0 3.1415" xyz="0 0 0"/>
       <xacro:frame_color/>
     </visual>
@@ -107,5 +107,5 @@
         <mesh filename="package://inmoov_description/meshes/ring3_2.stl" scale="0.001 0.001 0.001"/>
       </geometry>
-      <origin rpy="0 0 0" xyz="0 0 0"/>
+      <origin rpy="0 0 3.1415" xyz="0 0 0"/>
       <xacro:frame_color/>
     </visual>
@@ -116,5 +116,5 @@
         <mesh filename="package://inmoov_description/meshes/ring3_3.stl" scale="0.001 0.001 0.001"/>
       </geometry>
-      <origin rpy="0 0 0" xyz="0 0 0"/>
+      <origin rpy="0 0 3.1415" xyz="0 0 0"/>
       <xacro:frame_color/>
     </visual>
@@ -125,5 +125,5 @@
         <mesh filename="package://inmoov_description/meshes/ring3_4.stl" scale="0.001 0.001 0.001"/>
       </geometry>
-      <origin rpy="0 0 0" xyz="0 0 0"/>
+      <origin rpy="0 0 3.1415" xyz="0 0 0"/>
       <xacro:frame_color/>
     </visual>
@@ -134,5 +134,5 @@
         <mesh filename="package://inmoov_description/meshes/${side}_pinky3_1.stl" scale="0.001 0.001 0.001"/>
       </geometry>
-      <origin rpy="0 0 0" xyz="0 0 0"/>
+      <origin rpy="0 0 3.1415" xyz="0 0 0"/>
       <xacro:frame_color/>
     </visual>
@@ -143,5 +143,5 @@
         <mesh filename="package://inmoov_description/meshes/pinky3_2.stl" scale="0.001 0.001 0.001"/>
       </geometry>
-      <origin rpy="0 0 0" xyz="0 0 0"/>
+      <origin rpy="0 0 3.1415" xyz="0 0 0"/>
       <xacro:frame_color/>
     </visual>
@@ -152,5 +152,5 @@
         <mesh filename="package://inmoov_description/meshes/pinky3_3.stl" scale="0.001 0.001 0.001"/>
       </geometry>
-      <origin rpy="0 0 0" xyz="0 0 0"/>
+      <origin rpy="0 0 3.1415" xyz="0 0 0"/>
       <xacro:frame_color/>
     </visual>
@@ -161,5 +161,5 @@
         <mesh filename="package://inmoov_description/meshes/pinky3_4.stl" scale="0.001 0.001 0.001"/>
       </geometry>
-      <origin rpy="0 0 0" xyz="0 0 0"/>
+      <origin rpy="0 0 3.1415" xyz="0 0 0"/>
       <xacro:frame_color/>
     </visual>
@@ -168,12 +168,13 @@
    <axis xyz="0 0 1"/>
    <limit effort="1000.0" lower="0" upper="${neg *1.57}" velocity="0.5"/>
-   <origin rpy="0 ${neg * 0.1} 0" xyz="${neg * -0.029} 0 -0.0577"/>
+   <origin rpy="3.1415 ${neg * 0.1} 0" xyz="${neg * -0.029} 0 -0.0577"/>
+   <mimic joint="${side}_thumb" multiplier="${neg *-0.75}" offset="0"/>
    <parent link="${side}_hand"/>
    <child link="${side}_thumb1"/>
   </joint>
-  <joint name="${side}_thumb2" type="revolute">
-   <axis xyz="1 0 0"/>
-<limit effort="1000.0" lower="-1.57" upper="0" velocity="0.5"/>
-    <origin rpy="0 ${neg * 0.82} 0" xyz="${neg * -0.0287} -0.0006 -0.0123"/>
+  <joint name="${side}_thumb" type="revolute">
+   <axis xyz="1 0 0"/>
+<limit effort="1000.0" lower="0" upper="1.5" velocity="0.5"/>
+    <origin rpy="0 ${neg * 2.3} ${neg * -0.3}" xyz="${neg * -0.02725} -0.0006 0.014"/>
     <parent link="${side}_thumb1"/>
     <child link="${side}_thumb2"/>
@@ -183,4 +184,5 @@
 <limit effort="1000.0" lower="-1.57" upper="0" velocity="0.5"/>
 <origin rpy="0 0 0" xyz="0 0 -0.035"/>
+    <mimic joint="${side}_thumb" multiplier="1" offset="0"/>
     <parent link="${side}_thumb2"/>
     <child link="${side}_thumb3"/>
@@ -188,12 +190,13 @@
   <joint name="${side}_index1" type="revolute">
    <axis xyz="1 0 0"/>
-<limit effort="1000.0" lower="-1.57" upper="0" velocity="0.5"/>
-<origin rpy="0 ${neg * 0.1} 0" xyz="${neg * -0.0342} -0.0015 -0.119"/>
+<limit effort="1000.0" lower="0" upper="1.5" velocity="0.5"/>
+<origin rpy="0 ${neg * -0.1} 3.1415" xyz="${neg * -0.0342} -0.0015 -0.119"/>
+    <mimic joint="${side}_index" multiplier="1" offset="0"/>
     <parent link="${side}_hand"/>
     <child link="${side}_index1"/>
   </joint>
-  <joint name="${side}_index2" type="revolute">
-   <axis xyz="1 0 0"/>
-<limit effort="1000.0" lower="-1.57" upper="0" velocity="0.5"/>
+  <joint name="${side}_index" type="revolute">
+   <axis xyz="1 0 0"/>
+<limit effort="1000.0" lower="0" upper="1.5" velocity="0.5"/>
 <origin rpy="0 0 0" xyz="0 0.001 -0.03595"/>
     <parent link="${side}_index1"/>
@@ -202,6 +205,7 @@
   <joint name="${side}_index3" type="revolute">
    <axis xyz="1 0 0"/>
-<limit effort="1000.0" lower="-1.57" upper="0" velocity="0.5"/>
+<limit effort="1000.0" lower="0" upper="1.5" velocity="0.5"/>
 <origin rpy="0 0 0" xyz="0 0 -0.024"/>
+    <mimic joint="${side}_index" multiplier="1" offset="0"/>
     <parent link="${side}_index2"/>
     <child link="${side}_index3"/>
@@ -209,12 +213,13 @@
   <joint name="${side}_middle1" type="revolute">
    <axis xyz="1 0 0"/>
-<limit effort="1000.0" lower="-1.57" upper="0" velocity="0.5"/>
-<origin rpy="0 0 0" xyz="${neg * -0.007} -0.00175 -0.12325"/>
+<limit effort="1000.0" lower="0" upper="1.5" velocity="0.5"/>
+<origin rpy="0 0 3.1415" xyz="${neg * -0.007} -0.00175 -0.12325"/>
+    <mimic joint="${side}_middle" multiplier="1" offset="0"/>
     <parent link="${side}_hand"/>
     <child link="${side}_middle1"/>
   </joint>
-  <joint name="${side}_middle2" type="revolute">
-   <axis xyz="1 0 0"/>
-<limit effort="1000.0" lower="-1.57" upper="0" velocity="0.5"/>
+  <joint name="${side}_middle" type="revolute">
+   <axis xyz="1 0 0"/>
+<limit effort="1000.0" lower="0" upper="1.5" velocity="0.5"/>
 <origin rpy="0 0 0" xyz="0 0.000 -0.0389"/>
     <parent link="${side}_middle1"/>
@@ -225,4 +230,5 @@
 <limit effort="1000.0" lower="-1.57" upper="0" velocity="0.5"/>
 <origin rpy="0 0 0" xyz="0 0.0005 -0.0259"/>
+    <mimic joint="${side}_middle" multiplier="1" offset="0"/>
     <parent link="${side}_middle2"/>
     <child link="${side}_middle3"/>
@@ -231,12 +237,13 @@
    <axis xyz="0 0 1"/>
 <limit effort="1000.0" lower="${neg *-1.57}" upper="0" velocity="0.5"/>
-<origin rpy="0 ${neg * 0.7} 0" xyz="${neg * 0.00705} 0 -0.0794"/>
+<origin rpy="0 ${neg * -0.7} 3.1415" xyz="${neg * 0.00705} 0 -0.0794"/>
+    <mimic joint="${side}_ring" multiplier="${neg * -0.1}" offset="0"/>
     <parent link="${side}_hand"/>
     <child link="${side}_ring1"/>
   </joint>
-  <joint name="${side}_ring2" type="revolute">
-   <axis xyz="1 0 0"/>
-<limit effort="1000.0" lower="-1.57" upper="0" velocity="0.5"/>
-<origin rpy="0 ${neg * -0.78} 0" xyz="${neg * 0.035} -.00125 -0.0167"/>
+  <joint name="${side}_ring" type="revolute">
+   <axis xyz="1 0 0"/>
+<limit effort="1000.0" lower="0" upper="1.5" velocity="0.5"/>
+<origin rpy="0 ${neg * 0.7775} 0" xyz="${neg * -0.0351} 0.00126 -0.0166"/>
     <parent link="${side}_ring1"/>
     <child link="${side}_ring2"/>
@@ -246,4 +253,5 @@
 <limit effort="1000.0" lower="-1.57" upper="0" velocity="0.5"/>
 <origin rpy="0 0 0" xyz="0 0.0005 -0.0345"/>
+    <mimic joint="${side}_ring" multiplier="1" offset="0"/>
     <parent link="${side}_ring2"/>
     <child link="${side}_ring3"/>
@@ -253,4 +261,5 @@
 <limit effort="1000.0" lower="-1.57" upper="0" velocity="0.5"/>
 <origin rpy="0 0 0" xyz="0 0.0004 -0.0229"/>
+    <mimic joint="${side}_ring" multiplier="1" offset="0"/>
     <parent link="${side}_ring3"/>
     <child link="${side}_ring4"/>
@@ -259,12 +268,13 @@
    <axis xyz="0 0 1"/>
 <limit effort="1000.0" lower="${neg *-1.57}" upper="0" velocity="0.5"/>
-<origin rpy="0 ${neg * 0.7} 0" xyz="${neg * 0.0270} 0 -0.0555"/>
+<origin rpy="0 ${neg * -0.7} 3.1415" xyz="${neg * 0.0270} 0 -0.0555"/>
+    <mimic joint="${side}_pinky" multiplier="${neg * -0.1}" offset="0"/>
     <parent link="${side}_hand"/>
     <child link="${side}_pinky1"/>
   </joint>
-  <joint name="${side}_pinky2" type="revolute">
-   <axis xyz="1 0 0"/>
-<limit effort="1000.0" lower="-1.57" upper="0" velocity="0.5"/>
-<origin rpy="0 ${neg * -0.93} 0" xyz="${neg * 0.046} 0 -0.0228"/>
+  <joint name="${side}_pinky" type="revolute">
+   <axis xyz="1 0 0"/>
+<limit effort="1000.0" lower="0" upper="1.5" velocity="0.5"/>
+<origin rpy="0 ${neg * 0.93} 0" xyz="${neg * -0.046} -0 -0.0228"/>
     <parent link="${side}_pinky1"/>
     <child link="${side}_pinky2"/>
@@ -274,4 +284,5 @@
 <limit effort="1000.0" lower="-1.57" upper="0" velocity="0.5"/>
 <origin rpy="0 0 0" xyz="0 0.0005 -0.031"/>
+    <mimic joint="${side}_pinky" multiplier="1" offset="0"/>
     <parent link="${side}_pinky2"/>
     <child link="${side}_pinky3"/>
@@ -281,4 +292,5 @@
 <limit effort="1000.0" lower="-1.57" upper="0" velocity="0.5"/>
 <origin rpy="0 0 0" xyz="0 0.0004 -0.0208"/>
+    <mimic joint="${side}_pinky" multiplier="1" offset="0"/>
     <parent link="${side}_pinky3"/>
     <child link="${side}_pinky4"/>
@@ -298,5 +310,5 @@
         <mesh filename="package://inmoov_description/meshes/${side}_cover_handring.stl" scale="0.001 0.001 0.001"/>
       </geometry>
-      <origin rpy="0 0 0" xyz="0 0 0"/>
+      <origin rpy="0 0 3.1415" xyz="0 0 0"/>
       <xacro:cover_color/>
     </visual>
@@ -307,5 +319,5 @@
         <mesh filename="package://inmoov_description/meshes/${side}_cover_handpinky.stl" scale="0.001 0.001 0.001"/>
       </geometry>
-      <origin rpy="0 0 0" xyz="0 0 0"/>
+      <origin rpy="0 0 3.1415" xyz="0 0 0"/>
       <xacro:cover_color/>
     </visual>
@@ -316,5 +328,5 @@
         <mesh filename="package://inmoov_description/meshes/${side}_cover_thumb.stl" scale="0.001 0.001 0.001"/>
       </geometry>
-      <origin rpy="0 0 0" xyz="0 0 0"/>
+      <origin rpy="3.1415 0 0" xyz="0 0 0"/>
       <xacro:cover_color/>
     </visual>
@@ -325,5 +337,5 @@
         <mesh filename="package://inmoov_description/meshes/${side}_cover_index.stl" scale="0.001 0.001 0.001"/>
       </geometry>
-      <origin rpy="0 0 0" xyz="0 0 0"/>
+      <origin rpy="0 0 3.1415" xyz="0 0 0"/>
       <xacro:cover_color/>
     </visual>
@@ -334,5 +346,5 @@
         <mesh filename="package://inmoov_description/meshes/${side}_cover_middle.stl" scale="0.001 0.001 0.001"/>
       </geometry>
-      <origin rpy="0 0 0" xyz="0 0 0"/>
+      <origin rpy="0 0 3.1415" xyz="0 0 0"/>
       <xacro:cover_color/>
     </visual>
@@ -343,5 +355,5 @@
         <mesh filename="package://inmoov_description/meshes/${side}_cover_ring.stl" scale="0.001 0.001 0.001"/>
       </geometry>
-      <origin rpy="0 0 0" xyz="0 0 0"/>
+      <origin rpy="0 0 3.1415" xyz="0 0 0"/>
       <xacro:cover_color/>
     </visual>
@@ -352,5 +364,5 @@
         <mesh filename="package://inmoov_description/meshes/${side}_cover_pinky.stl" scale="0.001 0.001 0.001"/>
       </geometry>
-      <origin rpy="0 0 0" xyz="0 0 0"/>
+      <origin rpy="0 0 3.1415" xyz="0 0 0"/>
       <xacro:cover_color/>
     </visual>
@@ -362,35 +374,35 @@
   </joint>
   <joint name="${side}_cover_handring" type="fixed">
-<origin rpy="0 ${neg * -0.7} 0" xyz="${neg * 0.015} 0.009 -0.0008"/>
+<origin rpy="0 ${neg * 0.7} 0" xyz="${neg * -0.015} -0.009 -0.0008"/>
     <parent link="${side}_ring1"/>
     <child link="${side}_cover_handring"/>
   </joint>
   <joint name="${side}_cover_handpinky" type="fixed">
-<origin rpy="0 ${neg * -0.7} 0" xyz="${neg * 0.0205} 0.01 -0.0069"/>
+<origin rpy="0 ${neg * 0.7} 0" xyz="${neg * -0.0205} -0.01 -0.0069"/>
     <parent link="${side}_pinky1"/>
     <child link="${side}_cover_handpinky"/>
   </joint>
   <joint name="${side}_cover_thumb" type="fixed">
-    <origin rpy="0 ${neg * 3.2} 0" xyz="${neg * -0.02125} 0.01 0.0047"/>
+    <origin rpy="0 ${neg * 3.1} 0" xyz="${neg * -0.02125} -0.01 -0.0047"/>
     <parent link="${side}_thumb1"/>
     <child link="${side}_cover_thumb"/>
   </joint>
   <joint name="${side}_cover_index" type="fixed">
-    <origin rpy="${neg * -0.05} 0 0" xyz="0 0.0071 -0.012"/>
+    <origin rpy="${neg * 0.05} 0 0" xyz="0 -0.0071 -0.012"/>
     <parent link="${side}_index1"/>
     <child link="${side}_cover_index"/>
   </joint>
   <joint name="${side}_cover_middle" type="fixed">
-    <origin rpy="${neg * -0.05} 0 0" xyz="0 0.0071 -0.012"/>
+    <origin rpy="${neg * -0.05} 0 0" xyz="0 -0.0071 -0.012"/>
     <parent link="${side}_middle1"/>
     <child link="${side}_cover_middle"/>
   </joint>
   <joint name="${side}_cover_ring" type="fixed">
-    <origin rpy="${neg * -0.05} ${neg * 0.1} 0" xyz="0 0.0071 -0.011"/>
+    <origin rpy="${neg * -0.05} ${neg * -0.1} 0" xyz="0 -0.005 -0.011"/>
     <parent link="${side}_ring2"/>
     <child link="${side}_cover_ring"/>
   </joint>
   <joint name="${side}_cover_pinky" type="fixed">
-    <origin rpy="${neg * -0.05} ${neg * 0.1} 0" xyz="0 0.0071 -0.0105"/>
+    <origin rpy="${neg * -0.05} ${neg * -0.1} 0" xyz="0 -0.005 -0.0105"/>
     <parent link="${side}_pinky2"/>
     <child link="${side}_cover_pinky"/>

File: inmoov_description/urdf/asmHead.urdf.xacro (robot description, xacro)
@@ -26,5 +26,5 @@
         <mesh filename="package://inmoov_description/meshes/jaw.stl" scale="0.001 0.001 0.001"/>
       </geometry>
-      <origin rpy="0 0 0" xyz="0 0 0"/>
+      <origin rpy="0 0 3.1415" xyz="0 0 0"/>
       <xacro:cover_color/>
     </visual>
@@ -59,15 +59,15 @@
   <joint name="head_leftright" type="revolute">
    <axis xyz="0 0 1"/>
-<limit effort="1000.0" lower="-1.57" upper="1.57" velocity="0.5"/>
-<origin rpy="0 0 0" xyz="0 0 0.0245"/>
-    <parent link="head_base"/>
-    <child link="head"/>
+   <limit effort="1000.0" lower="-1.57" upper="1.57" velocity="0.5"/>
+   <origin rpy="0 0 0" xyz="0 0 0.0245"/>
+   <parent link="head_base"/>
+   <child link="head"/>
   </joint>
   <joint name="jaw" type="revolute">
    <axis xyz="1 0 0"/>
-<limit effort="1000.0" lower="0" upper="-0.15" velocity="0.5"/>
-<origin rpy="-0.085 0 0" xyz="-0.001 0.0375 0.0437"/>
-    <parent link="head"/>
-    <child link="jaw"/>
+   <limit effort="1000.0" lower="0" upper="0.15" velocity="0.5"/>
+   <origin rpy="0.085 0 3.1415" xyz="-0.001 0.0375 0.0437"/>
+   <parent link="head"/>
+   <child link="jaw"/>
   </joint>
   <joint name="skull" type="fixed">
