Commit message: Update inmoov_description
update urdf definitions for inmoov; corrected joint orientation to match robot; added launch files

File: inmoov_description/robots/inmoov.urdf (robot description, URDF)
Before this commit: robot inmoov, 87 links, 86 joints
Links:
- removed link kinect
- added link kinect2_ir_optical_frame; visual mesh filename=package://inmoov_description/meshes/kinectone.stl scale=0.001 0.001 0.001
- added link kinect2_link; visual mesh filename=package://inmoov_description/meshes/kinectone.stl scale=0.001 0.001 0.001
- added link kinect2_rgb_optical_frame; visual mesh filename=package://inmoov_description/meshes/kinectone.stl scale=0.001 0.001 0.001
Joints:
- removed joint kinect
- added joint kinect2: type fixed, parent torso, child kinect2_link, origin xyz=0 0 0.066 rpy=-1.57 0 -1.57
- added joint kinect2_ir_optical_frame: type fixed, parent torso, child kinect2_ir_optical_frame, origin xyz=0 0 0.066 rpy=-1.57 0 -1.57
- added joint kinect2_rgb_optical: type fixed, parent torso, child kinect2_rgb_optical_frame, origin xyz=0 0 0.066 rpy=-1.57 0 -1.57
- joint chestplate: origin xyz=0 0.039 0.025 rpy=0 0 0 -> xyz=0.039 0 0.025 rpy=0 0 0
- joint disk: origin xyz=0 0 0.09 rpy=0 0 0 -> xyz=0.046 0 0.09 rpy=0 0 0
- joint eye_leftright: origin xyz=0.033 0 -0.0036 rpy=0 0 0 -> xyz=0 0.033 -0.0036 rpy=0 0 3.1415
- joint eyes_updown: axis 1 0 0 -> 0 1 0; origin xyz=0 0 0 rpy=0 0 0 -> xyz=0 0 0 rpy=0 0 3.1415
- joint face: origin xyz=0 0.0637 0.079 rpy=0 0 0 -> xyz=0.0637 0 0.079 rpy=0 0 0
- joint head_tilt: axis 0 1 0 -> 1 0 0; limit lower=-0.30 upper=0.30 effort=1000.0 velocity=0.5 -> lower=0.30 upper=-0.30 effort=1000.0 velocity=0.5; origin xyz=-0.001 -0.0315 0.4551 rpy=0 0 0 -> xyz=-0.0315  -0.001 0.4551 rpy=0 0 3.1415
- joint head_updown: axis 1 0 0 -> 0 1 0; origin xyz=0 0 0 rpy=0 0 0 -> xyz=0 0 0 rpy=0 0 3.1415
- joint jaw: origin xyz=-0.001 0.0375 0.0437 rpy=0.085 0 3.1415 -> xyz=0.0375 0.0005 0.0437 rpy=0 -0.09 3.1415
- joint left_bicep: origin xyz=0 -0.0278 -0.2235 rpy=0 0 0 -> xyz=0 -0.0278 -0.2235 rpy=0 0.0 0
- joint left_bicep_rotate: origin xyz=-0.066 0 -0.060 rpy=0 0 0 -> xyz=-0.066 0 -0.060 rpy=0 0.0 0
- joint left_camera: origin xyz=0 -0.001 0 rpy=0 0 0 -> xyz=-0.001 0 0 rpy=0 0 0
- joint left_ear: origin xyz=-0.056 0.035 0.0437 rpy=0 0 0 -> xyz=0.035 0.056 0.0437 rpy=0 0 0
- joint left_eye: origin xyz=0 0.003 0 rpy=0 0 0 -> xyz=0.003 0 0 rpy=0 0 0
- joint left_eye_leftright: origin xyz=-0.033 0 -0.0036 rpy=0 0 0 -> xyz=0 -0.033 -0.0036 rpy=0 0 3.1415
- joint left_iris: origin xyz=0 0.0061 0 rpy=0 0 0 -> xyz=0.0061 0 0 rpy=0 0 0
- joint left_shoulder_side: origin xyz=-0.143 0 0.298 rpy=0 0 0 -> xyz=0 0.143 0.298 rpy=0 0 -1.57
- joint left_shoulder_up: origin xyz=-0.012 0 -0.04 rpy=0 0 0 -> xyz=-0.012 0 -0.04 rpy=0 0 0.0
- joint right_bicep: origin xyz=0 -0.0278 -0.2235 rpy=0 0 0 -> xyz=0 -0.0278 0.2235 rpy=0 3.14 0
- joint right_bicep_rotate: origin xyz=0.066 0 -0.060 rpy=0 0 0 -> xyz=0.066 0 -0.060 rpy=0 3.14 0
- joint right_camera: origin xyz=0 -0.001 0 rpy=0 0 0 -> xyz=-0.001 0 0 rpy=0 0 0
- joint right_ear: origin xyz=0.056 0.035 0.0437 rpy=0 0 0 -> xyz=0.035 -0.056 0.0437 rpy=0 0 0
- joint right_eye: origin xyz=0 0.003 0 rpy=0 0 0 -> xyz=0.003 0 0 rpy=0 0 0
- joint right_iris: origin xyz=0 0.0061 0 rpy=0 0 0 -> xyz=0.0061 0 0 rpy=0 0 0
- joint right_shoulder_side: limit lower=-0.75 upper=0 effort=1000.0 velocity=0.5 -> lower=0 upper=0.75 effort=1000.0 velocity=0.5; origin xyz=0.143 0 0.298 rpy=0 0 0 -> xyz=0 -0.143 0.298 rpy=0 0 1.57
- joint right_shoulder_up: origin xyz=0.012 0 -0.04 rpy=0 0 0 -> xyz=-0.012 0 -0.04 rpy=0 0 3.14
- joint skull: origin xyz=-0.001 0.044 -0.0245 rpy=0 0 0 -> xyz=0.044 0 -0.0245 rpy=0 0 0
- joint waist_lean: axis 0 1 0 -> 1 0 0

File: inmoov_description/robots/inmoov.urdf.xacro (robot description, xacro)
@@ -36,5 +36,5 @@
         <mesh filename="package://inmoov_description/meshes/virtual.stl" scale="0.001 0.001 0.001"/>
       </geometry>
-      <origin rpy="0 0 0" xyz="0 0 0"/>
+      <origin rpy="0 0 3.1415" xyz="0 0 0"/>
       <xacro:frame_color/>
     </visual>
@@ -47,14 +47,14 @@
   <xacro:torso side="right" covers="yes" />
   <joint name="head_tilt" type="revolute">
-   <axis xyz="0 1 0"/>
-   <limit effort="1000.0" lower="-0.30" upper="0.30" velocity="0.5"/>
-   <origin rpy="0 0 0" xyz="-0.001 -0.0315 0.4551"/>
+   <axis xyz="1 0 0"/>
+   <limit effort="1000.0" lower="0.30" upper="-0.30" velocity="0.5"/>
+   <origin rpy="0 0 3.1415" xyz="-0.0315  -0.001 0.4551"/>
    <parent link="torso"/>
    <child link="head_tilt"/>
   </joint>
   <joint name="head_updown" type="revolute">
-   <axis xyz="1 0 0"/>
+   <axis xyz="0 1 0"/>
    <limit effort="1000.0" lower="-0.30" upper="0.30" velocity="0.5"/>
-   <origin rpy="0 0 0" xyz="0 0 0"/>
+   <origin rpy="0 0 3.1415" xyz="0 0 0"/>
    <parent link="head_tilt"/>
    <child link="head_base"/>
@@ -63,5 +63,5 @@
   <xacro:face covers="yes" />
   <joint name="face" type="fixed">
-    <origin rpy="0 0 0" xyz="0 0.0637 0.079"/>
+    <origin rpy="0 0 0" xyz="0.0637 0 0.079"/>
     <parent link="skull"/>
     <child link="face"/>
@@ -70,6 +70,6 @@
   <joint name="right_shoulder_side" type="revolute">
    <axis xyz="0 1 0"/>
-   <limit effort="1000.0" lower="-0.75" upper="0" velocity="0.5"/>
-   <origin rpy="0 0 0" xyz="0.143 0 0.298"/>
+   <limit effort="1000.0" lower="0" upper="0.75" velocity="0.5"/>
+   <origin rpy="0 0 1.57" xyz="0 -0.143 0.298"/>
    <parent link="torso"/>
    <child link="right_shoulder_base"/>
@@ -87,5 +87,5 @@
    <axis xyz="0 1 0"/>
    <limit effort="1000.0" lower="0" upper="0.75" velocity="0.5"/>
-   <origin rpy="0 0 0" xyz="-0.143 0 0.298"/>
+   <origin rpy="0 0 -1.57" xyz="0 0.143 0.298"/>
    <parent link="torso"/>
    <child link="left_shoulder_base"/>

File: inmoov_description/robots/inmoov_face.urdf (robot description, URDF)
Before this commit: robot inmoov_hand, 11 links, 10 joints
Joints:
- removed joint right_eye_leftright
- added joint eye_leftright: type revolute, parent eyesupport, child right_eyesupport, origin xyz=0 0.033 -0.0036 rpy=0 0 0, axis 0 0 1, limit lower=-0.45 upper=0.45 effort=1000.0 velocity=0.5
- joint eyes_updown: limit lower=-1.57 upper=1.57 effort=1000.0 velocity=0.5 -> lower=-0.45 upper=0.45 effort=1000.0 velocity=0.5
- joint left_camera: origin xyz=0 -0.001 0 rpy=0 0 0 -> xyz=-0.001 0 0 rpy=0 0 0
- joint left_eye: origin xyz=0 0.003 0 rpy=0 0 0 -> xyz=0.003 0 0 rpy=0 0 0
- joint left_eye_leftright: limit lower=-1.57 upper=1.57 effort=1000.0 velocity=0.5 -> lower=-0.45 upper=0.45 effort=1000.0 velocity=0.5; mimic (none) -> joint=eye_leftright multiplier=1 offset=0; origin xyz=-0.033 0 -0.0036 rpy=0 0 0 -> xyz=0 -0.033 -0.0036 rpy=0 0 0
- joint left_iris: origin xyz=0 0.0061 0 rpy=0 0 0 -> xyz=0.0061 0 0 rpy=0 0 0
- joint right_camera: origin xyz=0 -0.001 0 rpy=0 0 0 -> xyz=-0.001 0 0 rpy=0 0 0
- joint right_eye: origin xyz=0 0.003 0 rpy=0 0 0 -> xyz=0.003 0 0 rpy=0 0 0
- joint right_iris: origin xyz=0 0.0061 0 rpy=0 0 0 -> xyz=0.0061 0 0 rpy=0 0 0

File: inmoov_description/robots/inmoov_right_hand.urdf (robot description, URDF)
Before this commit: robot inmoov_hand, 27 links, 26 joints
Joints:
- joint right_pinky1: mimic joint=right_pinky multiplier=0.1 offset=0 -> joint=right_pinky multiplier=-0.1 offset=0
- joint right_ring1: mimic joint=right_ring multiplier=0.1 offset=0 -> joint=right_ring multiplier=-0.1 offset=0

File: inmoov_description/urdf/asmArm.urdf.xacro (robot description, xacro)
@@ -8,5 +8,5 @@
         <mesh filename="package://inmoov_description/meshes/${side}_shoulder_base.stl" scale="0.001 0.001 0.001"/>
       </geometry>
-      <origin rpy="0 0 0" xyz="0 0 0"/>
+      <origin rpy="0 0 ${(flip * 1.57) + 1.57}" xyz="0 0 0"/>
       <xacro:frame_color/>
     </visual>
@@ -26,5 +26,5 @@
         <mesh filename="package://inmoov_description/meshes/bicep.stl" scale="0.001 0.001 0.001"/>
       </geometry>
-      <origin rpy="0 0 0" xyz="0 0 0"/>
+      <origin rpy="0 ${(flip * 1.57) + 1.57)} 0" xyz="0 0 0"/>
       <xacro:frame_color/>
     </visual>
@@ -35,5 +35,5 @@
         <mesh filename="package://inmoov_description/meshes/bicepcover.stl" scale="0.001 0.001 0.001"/>
       </geometry>
-      <origin rpy="0 0 0" xyz="0 0 0"/>
+      <origin rpy="0 ${(flip * 1.57) + 1.57)} 0" xyz="0 0 0"/>
       <xacro:cover_color/>
     </visual>
@@ -51,5 +51,5 @@
     <axis xyz="1 0 0"/>
     <limit effort="1000.0" lower="0" upper="3.14" velocity="0.5"/>
-    <origin rpy="0 0 0" xyz="${flip * 0.012} 0 -0.04"/>
+    <origin rpy="0 0 ${(flip * 1.57) + 1.57}" xyz="-0.012 0 -0.04"/>
     <parent link="${side}_shoulder_base"/>
     <child link="${side}_shoulder"/>
@@ -58,5 +58,5 @@
     <axis xyz="0 0 1"/>
     <limit effort="1000.0" lower="-1.57" upper="1.57" velocity="0.5"/>
-    <origin rpy="0 0 0" xyz="${flip * 0.066} 0 -0.060"/>
+    <origin rpy="0 ${(flip * 1.57) + 1.57)} 0" xyz="${flip * 0.066} 0 -0.060"/>
     <parent link="${side}_shoulder"/>
     <child link="${side}_bicep"/>
@@ -65,5 +65,5 @@
     <axis xyz="1 0 0"/>
     <limit effort="1000.0" lower="0.4" upper="1.57" velocity="0.5"/>
-    <origin rpy="0 0 0" xyz="0 -0.0278 -0.2235"/>
+    <origin rpy="0 ${(flip * 1.57) + 1.57)} 0" xyz="0 -0.0278 ${flip * 0.2235}"/>
     <parent link="${side}_bicep"/>
     <child link="${side}_forearm"/>

File: inmoov_description/urdf/asmFace.urdf.xacro (robot description, xacro)
@@ -13,7 +13,7 @@
   </link>
   <joint name="eyes_updown" type="revolute">
-   <axis xyz="1 0 0"/>
+   <axis xyz="0 1 0"/>
    <limit effort="1000.0" lower="-0.45" upper="0.45" velocity="0.5"/>
-   <origin rpy="0 0 0" xyz="0 0 0"/>
+   <origin rpy="0 0 3.1415" xyz="0 0 0"/>
    <parent link="face"/>
    <child link="eyesupport"/>
@@ -24,5 +24,5 @@
         <mesh filename="package://inmoov_description/meshes/eyesupport.stl" scale="0.001 0.001 0.001"/>
       </geometry>
-      <origin rpy="0 0 0" xyz="0 0 0"/>
+      <origin rpy="0 0 3.1415" xyz="0 0 0"/>
       <xacro:frame_color/>
     </visual>
@@ -32,5 +32,5 @@
    <axis xyz="0 0 1"/>
    <limit effort="1000.0" lower="-0.45" upper="0.45" velocity="0.5"/>
-   <origin rpy="0 0 0" xyz="0.033 0 -0.0036"/>
+   <origin rpy="0 0 3.1415" xyz="0 0.033 -0.0036"/>
    <parent link="eyesupport"/>
    <child link="right_eyesupport"/>
@@ -41,5 +41,5 @@
    <limit effort="1000.0" lower="-0.45" upper="0.45" velocity="0.5"/>
    <mimic joint="eye_leftright" multiplier="1" offset="0"/>
-   <origin rpy="0 0 0" xyz="-0.033 0 -0.0036"/>
+   <origin rpy="0 0 3.1415" xyz="0 -0.033 -0.0036"/>
    <parent link="eyesupport"/>
    <child link="left_eyesupport"/>
@@ -84,15 +84,15 @@
   </link>
   <joint name="${side}_camera" type="fixed">
-    <origin rpy="0 0 0" xyz="0 -0.001 0"/>
+    <origin rpy="0 0 0" xyz="-0.001 0 0"/>
     <parent link="${side}_eyesupport"/>
     <child link="${side}_camera"/>
   </joint>
   <joint name="${side}_eye" type="fixed">
-    <origin rpy="0 0 0" xyz="0 0.003 0"/>
+    <origin rpy="0 0 0" xyz="0.003 0 0"/>
     <parent link="${side}_eyesupport"/>
     <child link="${side}_eye"/>
   </joint>
   <joint name="${side}_iris" type="fixed">
-    <origin rpy="0 0 0" xyz="0 0.0061 0"/>
+    <origin rpy="0 0 0" xyz="0.0061 0 0"/>
     <parent link="${side}_eyesupport"/>
     <child link="${side}_iris"/>

File: inmoov_description/urdf/asmHead.urdf.xacro (robot description, xacro)
@@ -35,5 +35,5 @@
         <mesh filename="package://inmoov_description/meshes/skull.stl" scale="0.001 0.001 0.001"/>
       </geometry>
-      <origin rpy="0 0 0" xyz="0.001 0 0"/>
+      <origin rpy="0 0 0" xyz="0 0 0"/>
       <xacro:cover_color/>
     </visual>
@@ -67,20 +67,20 @@
    <axis xyz="1 0 0"/>
    <limit effort="1000.0" lower="0" upper="0.15" velocity="0.5"/>
-   <origin rpy="0.085 0 3.1415" xyz="-0.001 0.0375 0.0437"/>
+   <origin rpy="0 -0.09 3.1415" xyz="0.0375 0.0005 0.0437"/>
    <parent link="head"/>
    <child link="jaw"/>
   </joint>
   <joint name="skull" type="fixed">
-    <origin rpy="0 0 0" xyz="-0.001 0.044 -0.0245"/>
+    <origin rpy="0 0 0" xyz="0.044 0 -0.0245"/>
     <parent link="head"/>
     <child link="skull"/>
   </joint>
   <joint name="left_ear" type="fixed">
-    <origin rpy="0 0 0" xyz="-0.056 0.035 0.0437"/>
+    <origin rpy="0 0 0" xyz="0.035 0.056 0.0437"/>
     <parent link="head"/>
     <child link="left_ear"/>
   </joint>
   <joint name="right_ear" type="fixed">
-    <origin rpy="0 0 0" xyz="0.056 0.035 0.0437"/>
+    <origin rpy="0 0 0" xyz="0.035 -0.056 0.0437"/>
     <parent link="head"/>
     <child link="right_ear"/>

File: inmoov_description/urdf/asmTorso.urdf.xacro (robot description, xacro)
@@ -17,5 +17,5 @@
         <mesh filename="package://inmoov_description/meshes/disk.stl" scale="0.001 0.001 0.001"/>
       </geometry>
-      <origin rpy="0 0 0" xyz="0 0.046 0"/>
+      <origin rpy="0 0 0" xyz="0 0 0"/>
       <xacro:cover_color/>
     </visual>
@@ -39,10 +39,28 @@
     </visual>
   </link>
-  <link name="kinect">
+  <link name="kinect2_link">
     <visual>
       <geometry>
         <mesh filename="package://inmoov_description/meshes/kinectone.stl" scale="0.001 0.001 0.001"/>
       </geometry>
-      <origin rpy="0 0 0" xyz="0 0 0"/>
+      <origin rpy="1.57 0 0" xyz="0 0 0"/>
+      <xacro:kinect_color/>
+    </visual>
+  </link>
+  <link name="kinect2_ir_optical_frame">
+    <visual>
+      <geometry>
+        <mesh filename="package://inmoov_description/meshes/kinectone.stl" scale="0.001 0.001 0.001"/>
+      </geometry>
+      <origin rpy="1.57 0 0" xyz="0 0 0"/>
+      <xacro:kinect_color/>
+    </visual>
+  </link>
+  <link name="kinect2_rgb_optical_frame">
+    <visual>
+      <geometry>
+        <mesh filename="package://inmoov_description/meshes/kinectone.stl" scale="0.001 0.001 0.001"/>
+      </geometry>
+      <origin rpy="1.57 0 0" xyz="0 0 0"/>
       <xacro:kinect_color/>
     </visual>
@@ -65,10 +83,10 @@
   </joint>
   <joint name="disk" type="fixed">
-      <origin rpy="0 0 0" xyz="0 0 0.09"/>
+      <origin rpy="0 0 0" xyz="0.046 0 0.09"/>
     <parent link="top_stomach"/>
     <child link="disk"/>
   </joint>
   <joint name="waist_lean" type="revolute">
-   <axis xyz="0 1 0"/>
+   <axis xyz="1 0 0"/>
 <limit effort="1000.0" lower="-0.30" upper="0.30" velocity="0.5"/>
 <origin rpy="0 0 0" xyz="0 0 0.11"/>
@@ -77,12 +95,22 @@
   </joint>
   <joint name="chestplate" type="fixed">
-<origin rpy="0 0 0" xyz="0 0.039 0.025"/>
+<origin rpy="0 0 0" xyz="0.039 0 0.025"/>
     <parent link="torso"/>
     <child link="chestplate"/>
   </joint>
-  <joint name="kinect" type="fixed">
-<origin rpy="0 0 0" xyz="0 0 0.066"/>
+  <joint name="kinect2" type="fixed">
+<origin rpy="-1.57 0 -1.57" xyz="0 0 0.066"/>
     <parent link="torso"/>
-    <child link="kinect"/>
+    <child link="kinect2_link"/>
+  </joint>
+  <joint name="kinect2_ir_optical_frame" type="fixed">
+<origin rpy="-1.57 0 -1.57" xyz="0 0 0.066"/>
+    <parent link="torso"/>
+    <child link="kinect2_ir_optical_frame"/>
+  </joint>
+  <joint name="kinect2_rgb_optical" type="fixed">
+<origin rpy="-1.57 0 -1.57" xyz="0 0 0.066"/>
+    <parent link="torso"/>
+    <child link="kinect2_rgb_optical_frame"/>
   </joint>
 </xacro:macro>
