Commit message: urdf updates
urdf updated with bringup joint names, stls and joints oriented x as forward, joints unflipped to native axis orientation

File: inmoov_description/robots/inmoov.urdf.xacro (robot description, xacro)
@@ -5,4 +5,5 @@
   <xacro:include filename="$(find inmoov_description)/urdf/asmTorso.urdf.xacro" />
   <xacro:include filename="$(find inmoov_description)/urdf/asmHead.urdf.xacro" />
+  <xacro:include filename="$(find inmoov_description)/urdf/asmEye.urdf.xacro" />
   <xacro:include filename="$(find inmoov_description)/urdf/asmFace.urdf.xacro" />
   <xacro:include filename="$(find inmoov_description)/urdf/asmArm.urdf.xacro" />
@@ -17,10 +18,10 @@
     </visual>
   </link>
-  <joint name="base_to_pedestal" type="fixed">
+  <joint name="base_to_pedestal_link" type="fixed">
     <parent link="base_link"/>
-    <child link="pedestal"/>
+    <child link="pedestal_link"/>
     <origin rpy="0 0 0"  xyz="0 0 0"/>
   </joint>
-  <link name="pedestal">
+  <link name="pedestal_link">
     <visual>
       <geometry>
@@ -31,5 +32,5 @@
     </visual>
   </link>
-  <link name="head_tilt">
+  <link name="head_tilt_link">
     <visual>
       <geometry>
@@ -40,62 +41,62 @@
     </visual>
   </link>
-  <joint name="pedestal_to_mid_stomach" type="fixed">
-    <parent link="pedestal"/>
-    <child link="mid_stomach"/>
+  <joint name="pedestal_to_mid_stomach_joint" type="fixed">
+    <parent link="pedestal_link"/>
+    <child link="mid_stomach_link"/>
      <origin rpy="0 0 0"  xyz="0 0 0"/>
   </joint>
-  <xacro:torso side="right" covers="yes" />
-  <joint name="head_tilt" type="revolute">
+  <xacro:torso covers="yes" />
+  <joint name="head_roll_link" type="revolute">
    <axis xyz="1 0 0"/>
    <limit effort="1000.0" lower="0.30" upper="-0.30" velocity="0.5"/>
    <origin rpy="0 0 3.1415" xyz="-0.0315  -0.001 0.4551"/>
-   <parent link="torso"/>
-   <child link="head_tilt"/>
+   <parent link="torso_link"/>
+   <child link="head_tilt_link"/>
   </joint>
-  <joint name="head_updown" type="revolute">
+  <joint name="head_tilt_link" type="revolute">
    <axis xyz="0 1 0"/>
    <limit effort="1000.0" lower="-0.30" upper="0.30" velocity="0.5"/>
    <origin rpy="0 0 3.1415" xyz="0 0 0"/>
-   <parent link="head_tilt"/>
-   <child link="head_base"/>
+   <parent link="head_tilt_link"/>
+   <child link="head_base_link"/>
   </joint>
   <xacro:head covers="yes" />
   <xacro:face covers="yes" />
-  <joint name="face" type="fixed">
+  <joint name="face_joint" type="fixed">
     <origin rpy="0 0 0" xyz="0.0637 0 0.079"/>
-    <parent link="skull"/>
-    <child link="face"/>
+    <parent link="skull_link"/>
+    <child link="face_link"/>
   </joint>
-  <xacro:arm side="right" flip="1" covers="yes" />
-  <joint name="right_shoulder_side" type="revolute">
-   <axis xyz="0 1 0"/>
-   <limit effort="1000.0" lower="0" upper="0.75" velocity="0.5"/>
-   <origin rpy="0 0 1.57" xyz="0 -0.143 0.298"/>
-   <parent link="torso"/>
-   <child link="right_shoulder_base"/>
+  <xacro:arm side="r" flip="1" covers="yes" />
+  <joint name="r_shoulder_out_joint" type="revolute">
+   <axis xyz="1 0 0"/>
+   <limit effort="1000.0" lower="0" upper="-0.75" velocity="0.5"/>
+   <origin rpy="0 0 0" xyz="0 -0.143 0.298"/>
+   <parent link="torso_link"/>
+   <child link="r_shoulder_base_link"/>
   </joint>
-  <xacro:hand side="right" neg="1" flip="0" covers="yes" />
-  <joint name="right_hand" type="revolute">
+  <xacro:hand side="r" flip="1" covers="yes" />
+  <joint name="r_wrist_roll_joint" type="revolute">
    <axis xyz="0 0 1"/>
    <limit effort="1000.0" lower="-3.14" upper="0" velocity="0.5"/>
-   <origin rpy="0 0 0" xyz="-0.01 -0.0144 -0.2885"/>
-   <parent link="right_forearm"/>
-   <child link="right_hand"/>
+   <origin rpy="0 0 0" xyz="-0.0144 0.01  -0.2885"/>
+   <parent link="r_forearm_link"/>
+   <child link="r_hand_link"/>
   </joint>
-  <xacro:arm side="left" flip="-1" covers="yes" />
-  <joint name="left_shoulder_side" type="revolute">
-   <axis xyz="0 1 0"/>
+  <xacro:arm side="l" flip="-1" covers="yes" />
+  <joint name="l_shoulder_out_joint" type="revolute">
+   <axis xyz="1 0 0"/>
    <limit effort="1000.0" lower="0" upper="0.75" velocity="0.5"/>
-   <origin rpy="0 0 -1.57" xyz="0 0.143 0.298"/>
-   <parent link="torso"/>
-   <child link="left_shoulder_base"/>
+   <origin rpy="0 0 0" xyz="0 0.143 0.298"/>
+   <parent link="torso_link"/>
+   <child link="l_shoulder_base_link"/>
   </joint>
-  <xacro:hand side="left" neg="-1" flip="3.1415926539" covers="yes" />
-  <joint name="left_hand" type="revolute">
+  <xacro:hand side="l" flip="-1" covers="yes" />
+  <joint name="l_wrist_roll_joint" type="revolute">
    <axis xyz="0 0 1"/>
    <limit effort="1000.0" lower="0" upper="3.14" velocity="0.5"/>
-   <origin rpy="0 0 0" xyz="0.01 -0.0144 -0.2885"/>
-   <parent link="left_forearm"/>
-   <child link="left_hand"/>
+   <origin rpy="0 0 0" xyz="-0.0144 -0.01  -0.2885"/>
+   <parent link="l_forearm_link"/>
+   <child link="l_hand_link"/>
   </joint>
 </robot>

File: inmoov_description/robots/inmoov_right_hand.urdf.xacro (robot description, xacro)
@@ -1,4 +1,5 @@
 <?xml version="1.0"?>
 <robot name="inmoov_hand" xmlns:xacro="http://ros.org/wiki/xacro">
+<xacro:include filename="$(find inmoov_description)/urdf/config.urdf.xacro" />
 <xacro:include filename="$(find inmoov_description)/urdf/materials.urdf.xacro" />
 <xacro:include filename="$(find inmoov_description)/urdf/asmHand.urdf.xacro" />
@@ -14,11 +15,11 @@
     </visual>
   </link>
-  <xacro:hand side="right" neg="1" flip="0" covers="yes" />
-  <joint name="base_to_hand" type="revolute">
+  <xacro:hand side="r" flip="1" covers="yes" />
+  <joint name="base_to_hand_joint" type="revolute">
    <axis xyz="0 0 1"/>
 <limit effort="1000.0" lower="-3.14" upper="0" velocity="0.5"/>
-<origin rpy="0 3.1415 0" xyz="0 0 0"/>
+<origin rpy="0 0 0" xyz="0 0 0"/>
     <parent link="base_link"/>
-    <child link="right_hand"/>
+    <child link="r_hand_link"/>
   </joint>
 </robot>

File: inmoov_description/urdf/asmArm.urdf.xacro (robot description, xacro)
@@ -3,14 +3,14 @@
 <xacro:include filename="$(find inmoov_description)/urdf/materials.urdf.xacro" />
 <xacro:macro name="arm" params="side flip covers">
-  <link name="${side}_shoulder_base">
+  <link name="${side}_shoulder_base_link">
     <visual>
       <geometry>
         <mesh filename="package://inmoov_meshes/meshes/${side}_shoulder_base.stl" scale="0.001 0.001 0.001"/>
       </geometry>
-      <origin rpy="0 0 ${(flip * 1.57) + 1.57}" xyz="0 0 0"/>
+      <origin rpy="0 0 0" xyz="0 0 0"/>
       <xacro:frame_color/>
     </visual>
   </link>
-  <link name="${side}_shoulder">
+  <link name="${side}_shoulder_link">
     <visual>
       <geometry>
@@ -21,23 +21,23 @@
     </visual>
   </link>
-  <link name="${side}_bicep">
+  <link name="${side}_bicep_link">
     <visual>
       <geometry>
         <mesh filename="package://inmoov_meshes/meshes/bicep.stl" scale="0.001 0.001 0.001"/>
       </geometry>
-      <origin rpy="0 ${(flip * 1.57) + 1.57} 0" xyz="0 0 0"/>
+      <origin rpy="0 0 0" xyz="0 0 0"/>
       <xacro:frame_color/>
     </visual>
   </link>
-  <link name="${side}_bicepcover">
+  <link name="${side}_bicepcover_link">
     <visual>
       <geometry>
         <mesh filename="package://inmoov_meshes/meshes/bicepcover.stl" scale="0.001 0.001 0.001"/>
       </geometry>
-      <origin rpy="0 ${(flip * 1.57) + 1.57} 0" xyz="0 0 0"/>
+      <origin rpy="0 0 0" xyz="0 0 0"/>
       <xacro:cover_color/>
     </visual>
   </link>
-  <link name="${side}_forearm">
+  <link name="${side}_forearm_link">
     <visual>
       <geometry>
@@ -48,29 +48,29 @@
     </visual>
   </link>
-  <joint name="${side}_shoulder_up" type="revolute">
-    <axis xyz="1 0 0"/>
-    <limit effort="1000.0" lower="0" upper="3.14" velocity="0.5"/>
-    <origin rpy="0 0 ${(flip * 1.57) + 1.57}" xyz="-0.012 0 -0.04"/>
-    <parent link="${side}_shoulder_base"/>
-    <child link="${side}_shoulder"/>
+  <joint name="${side}_shoulder_lift_joint" type="revolute">
+    <axis xyz="0 1 0"/>
+    <limit effort="1000.0" lower="0.7" upper="-2.5" velocity="0.5"/>
+    <origin rpy="0 0 0" xyz="0 ${flip * -0.012} -0.04"/>
+    <parent link="${side}_shoulder_base_link"/>
+    <child link="${side}_shoulder_link"/>
   </joint>
-  <joint name="${side}_bicep_rotate" type="revolute">
+  <joint name="${side}_upper_arm_roll_joint" type="revolute">
     <axis xyz="0 0 1"/>
     <limit effort="1000.0" lower="-1.57" upper="1.57" velocity="0.5"/>
-    <origin rpy="0 ${(flip * 1.57) + 1.57} 0" xyz="${flip * 0.066} 0 -0.060"/>
-    <parent link="${side}_shoulder"/>
-    <child link="${side}_bicep"/>
+    <origin rpy="0 0 0" xyz="0 ${flip * -0.066} -0.060"/>
+    <parent link="${side}_shoulder_link"/>
+    <child link="${side}_bicep_link"/>
   </joint>
-  <joint name="${side}_bicep" type="revolute">
-    <axis xyz="1 0 0"/>
-    <limit effort="1000.0" lower="0.4" upper="1.57" velocity="0.5"/>
-    <origin rpy="0 ${(flip * 1.57) + 1.57} 0" xyz="0 -0.0278 ${flip * 0.2235}"/>
-    <parent link="${side}_bicep"/>
-    <child link="${side}_forearm"/>
+  <joint name="${side}_elbow_flex_joint" type="revolute">
+    <axis xyz="0 1 0"/>
+    <limit effort="1000.0" lower="-0.4" upper="-1.57" velocity="0.5"/>
+    <origin rpy="0 0 0" xyz="-0.0278 0 -0.2235"/>
+    <parent link="${side}_bicep_link"/>
+    <child link="${side}_forearm_link"/>
   </joint>
-  <joint name="${side}_bicepcover" type="fixed">
+  <joint name="${side}_bicepcover_joint" type="fixed">
     <origin rpy="0 0 0" xyz="0 0 0"/>
-    <parent link="${side}_bicep"/>
-    <child link="${side}_bicepcover"/>
+    <parent link="${side}_bicep_link"/>
+    <child link="${side}_bicepcover_link"/>
   </joint>
 </xacro:macro>

File: inmoov_description/urdf/asmFace.urdf.xacro (robot description, xacro)
@@ -2,6 +2,7 @@
 <robot name="inmoov" xmlns:xacro="http://ros.org/wiki/xacro">
 <xacro:include filename="$(find inmoov_description)/urdf/materials.urdf.xacro" />
+<xacro:include filename="$(find inmoov_description)/urdf/asmEye.urdf.xacro" />
 <xacro:macro name="face" params="covers">
-  <link name="face">
+  <link name="face_link">
     <visual>
       <geometry>
@@ -12,43 +13,15 @@
     </visual>
   </link>
-  <joint name="eyes_updown" type="revolute">
+  <joint name="eyes_tilt_joint" type="revolute">
    <axis xyz="0 1 0"/>
    <limit effort="1000.0" lower="-0.45" upper="0.45" velocity="0.5"/>
-   <origin rpy="0 0 3.1415" xyz="0 0 0"/>
-   <parent link="face"/>
-   <child link="eyesupport"/>
+   <origin rpy="0 0 0" xyz="0 0 0"/>
+   <parent link="face_link"/>
+   <child link="eyesupport_link"/>
   </joint>
-  <link name="eyesupport">
+  <link name="eyesupport_link">
     <visual>
       <geometry>
         <mesh filename="package://inmoov_meshes/meshes/eyesupport.stl" scale="0.001 0.001 0.001"/>
-      </geometry>
-      <origin rpy="0 0 3.1415" xyz="0 0 0"/>
-      <xacro:frame_color/>
-    </visual>
-  </link>
-<xacro:asmEye side="right" flip="1" />
-  <joint name="eye_leftright" type="revolute">
-   <axis xyz="0 0 1"/>
-   <limit effort="1000.0" lower="-0.45" upper="0.45" velocity="0.5"/>
-   <origin rpy="0 0 3.1415" xyz="0 0.033 -0.0036"/>
-   <parent link="eyesupport"/>
-   <child link="right_eyesupport"/>
-  </joint>
-<xacro:asmEye side="left" flip="-1" />
-  <joint name="left_eye_leftright" type="revolute">
-   <axis xyz="0 0 1"/>
-   <limit effort="1000.0" lower="-0.45" upper="0.45" velocity="0.5"/>
-   <mimic joint="eye_leftright" multiplier="1" offset="0"/>
-   <origin rpy="0 0 3.1415" xyz="0 -0.033 -0.0036"/>
-   <parent link="eyesupport"/>
-   <child link="left_eyesupport"/>
-  </joint>
-</xacro:macro>
-<xacro:macro name="asmEye" params="side flip">
-  <link name="${side}_eyesupport">
-    <visual>
-      <geometry>
-        <mesh filename="package://inmoov_meshes/meshes/${side}_eyesupport.stl" scale="0.001 0.001 0.001"/>
       </geometry>
       <origin rpy="0 0 0" xyz="0 0 0"/>
@@ -56,45 +29,20 @@
     </visual>
   </link>
-  <link name="${side}_camera">
-    <visual>
-      <geometry>
-        <mesh filename="package://inmoov_meshes/meshes/camera.stl" scale="0.001 0.001 0.001"/>
-      </geometry>
-      <origin rpy="0 0 0" xyz="0 0 0"/>
-      <xacro:camera_color/>
-    </visual>
-  </link>
-  <link name="${side}_eye">
-    <visual>
-      <geometry>
-        <mesh filename="package://inmoov_meshes/meshes/eye.stl" scale="0.001 0.001 0.001"/>
-      </geometry>
-      <origin rpy="0 0 0" xyz="0 0 0"/>
-      <xacro:eyeball_color/>
-    </visual>
-  </link>
-  <link name="${side}_iris">
-    <visual>
-      <geometry>
-        <mesh filename="package://inmoov_meshes/meshes/iris.stl" scale="0.001 0.001 0.001"/>
-      </geometry>
-      <origin rpy="0 0 0" xyz="0 0 0"/>
-      <xacro:iris_color/>
-    </visual>
-  </link>
-  <joint name="${side}_camera" type="fixed">
-    <origin rpy="0 0 0" xyz="-0.001 0 0"/>
-    <parent link="${side}_eyesupport"/>
-    <child link="${side}_camera"/>
+<xacro:asmEye side="r"/>
+  <joint name="eyes_pan_joint" type="revolute">
+   <axis xyz="0 0 1"/>
+   <limit effort="1000.0" lower="-0.45" upper="0.45" velocity="0.5"/>
+   <origin rpy="0 0 0" xyz="0 0.033 -0.0036"/>
+   <parent link="eyesupport_link"/>
+   <child link="r_eyesupport_link"/>
   </joint>
-  <joint name="${side}_eye" type="fixed">
-    <origin rpy="0 0 0" xyz="0.003 0 0"/>
-    <parent link="${side}_eyesupport"/>
-    <child link="${side}_eye"/>
-  </joint>
-  <joint name="${side}_iris" type="fixed">
-    <origin rpy="0 0 0" xyz="0.0061 0 0"/>
-    <parent link="${side}_eyesupport"/>
-    <child link="${side}_iris"/>
+<xacro:asmEye side="l" />
+  <joint name="l_eye_pan_joint" type="revolute">
+   <axis xyz="0 0 1"/>
+   <limit effort="1000.0" lower="-0.45" upper="0.45" velocity="0.5"/>
+   <mimic joint="eyes_pan_joint" multiplier="1" offset="0"/>
+   <origin rpy="0 0 0" xyz="0 -0.033 -0.0036"/>
+   <parent link="eyesupport_link"/>
+   <child link="l_eyesupport_link"/>
   </joint>
 </xacro:macro>
