Commit message: urdf joint vars now defined from config.yaml
not the most elegant solution, but joint limits and velocity are set through config.yaml

File: inmoov_description/robots/inmoov.urdf.xacro (robot description, xacro)
@@ -1,4 +1,6 @@
 <?xml version="1.0"?>
 <robot name="inmoov" xmlns:xacro="http://ros.org/wiki/xacro">
+<xacro:include filename="$(find inmoov_description)/urdf/materials.urdf.xacro" />
+<xacro:include filename="$(find inmoov_description)/urdf/config.urdf.xacro" />
   <xacro:include filename="$(find inmoov_description)/urdf/materials.urdf.xacro" />
   <xacro:include filename="$(find inmoov_description)/urdf/asmBase.urdf.xacro" />
@@ -47,14 +49,14 @@
   </joint>
   <xacro:torso covers="yes" />
-  <joint name="head_roll_link" type="revolute">
+  <joint name="head_roll_joint" type="revolute">
    <axis xyz="1 0 0"/>
-   <limit effort="1000.0" lower="0.30" upper="-0.30" velocity="0.5"/>
+   <limit effort="1000.0" lower="${head_roll_joint_lower}" upper="${head_roll_joint_upper}" velocity="${head_roll_joint_velocity}" />
    <origin rpy="0 0 3.1415" xyz="-0.0315  -0.001 0.4551"/>
    <parent link="torso_link"/>
    <child link="head_tilt_link"/>
   </joint>
-  <joint name="head_tilt_link" type="revolute">
+  <joint name="head_tilt_joint" type="revolute">
    <axis xyz="0 1 0"/>
-   <limit effort="1000.0" lower="-0.30" upper="0.30" velocity="0.5"/>
+   <limit effort="1000.0" lower="${head_tilt_joint_lower}" upper="${head_tilt_joint_upper}" velocity="${head_tilt_joint_velocity}" />
    <origin rpy="0 0 3.1415" xyz="0 0 0"/>
    <parent link="head_tilt_link"/>
@@ -71,5 +73,5 @@
   <joint name="r_shoulder_out_joint" type="revolute">
    <axis xyz="1 0 0"/>
-   <limit effort="1000.0" lower="0" upper="-0.75" velocity="0.5"/>
+   <limit effort="1000.0" lower="${r_shoulder_out_joint_lower}" upper="${r_shoulder_out_joint_upper}" velocity="${r_shoulder_out_joint_velocity}" />
    <origin rpy="0 0 0" xyz="0 -0.143 0.298"/>
    <parent link="torso_link"/>
@@ -79,5 +81,5 @@
   <joint name="r_wrist_roll_joint" type="revolute">
    <axis xyz="0 0 1"/>
-   <limit effort="1000.0" lower="-3.14" upper="0" velocity="0.5"/>
+   <limit effort="1000.0" lower="${r_wrist_roll_joint_lower}" upper="${r_wrist_roll_joint_upper}" velocity="${r_wrist_roll_joint_velocity}" />
    <origin rpy="0 0 0" xyz="-0.0144 0.01  -0.2885"/>
    <parent link="r_forearm_link"/>
@@ -87,5 +89,5 @@
   <joint name="l_shoulder_out_joint" type="revolute">
    <axis xyz="1 0 0"/>
-   <limit effort="1000.0" lower="0" upper="0.75" velocity="0.5"/>
+   <limit effort="1000.0" lower="${l_shoulder_out_joint_lower}" upper="${l_shoulder_out_joint_upper}" velocity="${l_shoulder_out_joint_velocity}" />
    <origin rpy="0 0 0" xyz="0 0.143 0.298"/>
    <parent link="torso_link"/>
@@ -95,5 +97,5 @@
   <joint name="l_wrist_roll_joint" type="revolute">
    <axis xyz="0 0 1"/>
-   <limit effort="1000.0" lower="0" upper="3.14" velocity="0.5"/>
+   <limit effort="1000.0" lower="${l_wrist_roll_joint_lower}" upper="${l_wrist_roll_joint_upper}" velocity="${l_wrist_roll_joint_velocity}" />
    <origin rpy="0 0 0" xyz="-0.0144 -0.01  -0.2885"/>
    <parent link="l_forearm_link"/>

File: inmoov_description/robots/inmoov_face.urdf.xacro (robot description, xacro)
@@ -20,5 +20,5 @@
 <origin rpy="0 0 0" xyz="0 0 0"/>
     <parent link="base_link"/>
-    <child link="face"/>
+    <child link="face_link"/>
   </joint>
 </robot>

File: inmoov_description/robots/inmoov_head.urdf.xacro (robot description, xacro)
@@ -22,10 +22,10 @@
    <origin rpy="0 0 0" xyz="0 0 0"/>
    <parent link="base_link"/>
-   <child link="head_base"/>
+   <child link="head_base_link"/>
   </joint>
   <joint name="face" type="fixed">
     <origin rpy="0 0 0" xyz="0 0.0637 0.079"/>
-    <parent link="skull"/>
-    <child link="face"/>
+    <parent link="skull_link"/>
+    <child link="face_link"/>
   </joint>
 </robot>

File: inmoov_description/urdf/asmArm.urdf.xacro (robot description, xacro)
@@ -50,5 +50,10 @@
   <joint name="${side}_shoulder_lift_joint" type="revolute">
     <axis xyz="0 1 0"/>
-    <limit effort="1000.0" lower="0.7" upper="-2.5" velocity="0.5"/>
+    <xacro:if value="${side == 'l'}">
+      <limit effort="1000.0" lower="${l_shoulder_lift_joint_lower}" upper="${l_shoulder_lift_joint_upper}" velocity="${l_shoulder_lift_joint_velocity}" />
+    </xacro:if>
+    <xacro:if value="${side == 'r'}">
+      <limit effort="1000.0" lower="${r_shoulder_lift_joint_lower}" upper="${r_shoulder_lift_joint_upper}" velocity="${r_shoulder_lift_joint_velocity}" />
+    </xacro:if>
     <origin rpy="0 0 0" xyz="0 ${flip * -0.012} -0.04"/>
     <parent link="${side}_shoulder_base_link"/>
@@ -57,5 +62,10 @@
   <joint name="${side}_upper_arm_roll_joint" type="revolute">
     <axis xyz="0 0 1"/>
-    <limit effort="1000.0" lower="-1.57" upper="1.57" velocity="0.5"/>
+    <xacro:if value="${side == 'l'}">
+      <limit effort="1000.0" lower="${l_upper_arm_roll_joint_lower}" upper="${l_upper_arm_roll_joint_upper}" velocity="${l_upper_arm_roll_joint_velocity}" />
+    </xacro:if>
+    <xacro:if value="${side == 'r'}">
+      <limit effort="1000.0" lower="${r_upper_arm_roll_joint_lower}" upper="${r_upper_arm_roll_joint_upper}" velocity="${r_upper_arm_roll_joint_velocity}" />
+    </xacro:if>
     <origin rpy="0 0 0" xyz="0 ${flip * -0.066} -0.060"/>
     <parent link="${side}_shoulder_link"/>
@@ -64,5 +74,10 @@
   <joint name="${side}_elbow_flex_joint" type="revolute">
     <axis xyz="0 1 0"/>
-    <limit effort="1000.0" lower="-0.4" upper="-1.57" velocity="0.5"/>
+    <xacro:if value="${side == 'l'}">
+      <limit effort="1000.0" lower="${l_elbow_flex_joint_lower}" upper="${l_elbow_flex_joint_upper}" velocity="${l_elbow_flex_joint_velocity}" />
+    </xacro:if>
+    <xacro:if value="${side == 'r'}">
+      <limit effort="1000.0" lower="${r_elbow_flex_joint_lower}" upper="${r_elbow_flex_joint_upper}" velocity="${r_elbow_flex_joint_velocity}" />
+    </xacro:if>
     <origin rpy="0 0 0" xyz="-0.0278 0 -0.2235"/>
     <parent link="${side}_bicep_link"/>

File: inmoov_description/urdf/asmEye.urdf.xacro (robot description, xacro)
@@ -2,4 +2,5 @@
 <robot name="inmoov" xmlns:xacro="http://ros.org/wiki/xacro">
 <xacro:include filename="$(find inmoov_description)/urdf/materials.urdf.xacro" />
+<xacro:include filename="$(find inmoov_description)/urdf/config.urdf.xacro" />
 <xacro:macro name="asmEye" params="side">
   <link name="${side}_eyesupport_link">

File: inmoov_description/urdf/asmFace.urdf.xacro (robot description, xacro)
@@ -2,4 +2,5 @@
 <robot name="inmoov" xmlns:xacro="http://ros.org/wiki/xacro">
 <xacro:include filename="$(find inmoov_description)/urdf/materials.urdf.xacro" />
+<xacro:include filename="$(find inmoov_description)/urdf/config.urdf.xacro" />
 <xacro:include filename="$(find inmoov_description)/urdf/asmEye.urdf.xacro" />
 <xacro:macro name="face" params="covers">
@@ -15,5 +16,5 @@
   <joint name="eyes_tilt_joint" type="revolute">
    <axis xyz="0 1 0"/>
-   <limit effort="1000.0" lower="-0.45" upper="0.45" velocity="0.5"/>
+   <limit effort="1000.0" lower="${eyes_tilt_joint_lower}" upper="${eyes_tilt_joint_upper}" velocity="${eyes_tilt_joint_velocity}" />
    <origin rpy="0 0 0" xyz="0 0 0"/>
    <parent link="face_link"/>
@@ -32,5 +33,5 @@
   <joint name="eyes_pan_joint" type="revolute">
    <axis xyz="0 0 1"/>
-   <limit effort="1000.0" lower="-0.45" upper="0.45" velocity="0.5"/>
+    <limit effort="1000.0" lower="${eyes_pan_joint_lower}" upper="${eyes_pan_joint_upper}" velocity="${eyes_pan_joint_velocity}" />
    <origin rpy="0 0 0" xyz="0 0.033 -0.0036"/>
    <parent link="eyesupport_link"/>
@@ -40,5 +41,5 @@
   <joint name="l_eye_pan_joint" type="revolute">
    <axis xyz="0 0 1"/>
-   <limit effort="1000.0" lower="-0.45" upper="0.45" velocity="0.5"/>
+   <limit effort="1000.0" lower="${eyes_pan_joint_lower}" upper="${eyes_pan_joint_upper}" velocity="${eyes_pan_joint_velocity}" />
    <mimic joint="eyes_pan_joint" multiplier="1" offset="0"/>
    <origin rpy="0 0 0" xyz="0 -0.033 -0.0036"/>

File: inmoov_description/urdf/asmHand.urdf.xacro (robot description, xacro)
@@ -3,7 +3,5 @@
   xmlns:xacro="http://ros.org/wiki/xacro">
   <xacro:include filename="$(find inmoov_description)/urdf/materials.urdf.xacro" />
-  <xacro:include filename="$(find inmoov_bringup)/config/config.xacro" />
-  <xacro:property name="filename" value="$(find inmoov_bringup)/config/config.yaml"/>
-  <!--xacro:property name="p" value="${load_yaml(filename)}"/-->
+  <xacro:include filename="$(find inmoov_description)/urdf/config.urdf.xacro" />
   <xacro:macro name="hand" params="side flip covers">
     <link name="${side}_hand_link">
@@ -171,5 +169,10 @@
     <joint name="${side}_thumb1_joint" type="revolute">
       <axis xyz="0 0 1"/>
-      <limit effort="1000.0" lower="0" upper="${flip *-1.57}" velocity="0.5"/>
+        <xacro:if value="${side == 'l'}">
+          <limit effort="1000.0" lower="${l_thumb_joint_lower}" upper="${l_thumb_joint_upper}" velocity="${l_thumb_joint_velocity}" />
+        </xacro:if>
+        <xacro:if value="${side == 'r'}">
+          <limit effort="1000.0" lower="${r_thumb_joint_lower}" upper="${r_thumb_joint_upper}" velocity="${r_thumb_joint_velocity}" />
+        </xacro:if>
       <origin rpy="${flip * 0.1} 0 0" xyz="0 ${flip * 0.029} -0.0577"/>
       <mimic joint="${side}_thumb_joint" multiplier="${flip *0.75}" offset="0"/>
@@ -179,6 +182,10 @@
     <joint name="${side}_thumb_joint" type="revolute">
       <axis xyz="0 1 0"/>
-      <!--limit effort="1000.0" lower="${p['joints']['r_thumb_joint']['mingoal']}" upper="${p['joints']['r_thumb_joint']['maxgoal']}" velocity="${p['joints']['r_thumb_joint']['maxspeed']}"/-->
-      <limit effort="1000.0" lower="-0.1" upper="1.1" velocity="0.5"/>
+        <xacro:if value="${side == 'l'}">
+          <limit effort="1000.0" lower="${l_thumb_joint_lower}" upper="${l_thumb_joint_upper}" velocity="${l_thumb_joint_velocity}" />
+        </xacro:if>
+        <xacro:if value="${side == 'r'}">
+          <limit effort="1000.0" lower="${r_thumb_joint_lower}" upper="${r_thumb_joint_upper}" velocity="${r_thumb_joint_velocity}" />
+        </xacro:if>
       <origin rpy="${flip * 0.825} -0.1 ${flip * 0.3}" xyz="-0.00052 ${flip * 0.02725}  -0.013"/>
       <parent link="${side}_thumb1_link"/>
@@ -187,5 +194,10 @@
     <joint name="${side}_thumb3_joint" type="revolute">
       <axis xyz="0 1 0"/>
-      <limit effort="1000.0" lower="-1.57" upper="0" velocity="0.5"/>
+        <xacro:if value="${side == 'l'}">
+          <limit effort="1000.0" lower="${l_thumb_joint_lower}" upper="${l_thumb_joint_upper}" velocity="${l_thumb_joint_velocity}" />
+        </xacro:if>
+        <xacro:if value="${side == 'r'}">
+          <limit effort="1000.0" lower="${r_thumb_joint_lower}" upper="${r_thumb_joint_upper}" velocity="${r_thumb_joint_velocity}" />
+        </xacro:if>
       <origin rpy="0 0 0" xyz="0 0 -0.035"/>
       <mimic joint="${side}_thumb_joint" multiplier="1" offset="0"/>
@@ -195,5 +207,10 @@
     <joint name="${side}_index1_joint" type="revolute">
       <axis xyz="0 1 0"/>
-      <limit effort="1000.0" lower="0.1" upper="-1.5" velocity="0.5"/>
+        <xacro:if value="${side == 'l'}">
+          <limit effort="1000.0" lower="${l_index_joint_lower}" upper="${l_index_joint_upper}" velocity="${l_index_joint_velocity}" />
+        </xacro:if>
+        <xacro:if value="${side == 'r'}">
+          <limit effort="1000.0" lower="${r_index_joint_lower}" upper="${r_index_joint_upper}" velocity="${r_index_joint_velocity}" />
+        </xacro:if>
       <origin rpy="${flip * 0.1} 0 0" xyz="-0.0015 ${flip * 0.0342}  -0.119"/>
       <mimic joint="${side}_index_joint" multiplier="1" offset="0"/>
@@ -203,5 +220,10 @@
     <joint name="${side}_index_joint" type="revolute">
       <axis xyz="0 1 0"/>
-      <limit effort="1000.0" lower="-0.1" upper="1.5" velocity="0.5"/>
+        <xacro:if value="${side == 'l'}">
+          <limit effort="1000.0" lower="${l_index_joint_lower}" upper="${l_index_joint_upper}" velocity="${l_index_joint_velocity}" />
+        </xacro:if>
+        <xacro:if value="${side == 'r'}">
+          <limit effort="1000.0" lower="${r_index_joint_lower}" upper="${r_index_joint_upper}" velocity="${r_index_joint_velocity}" />
+        </xacro:if>
       <origin rpy="0 0 0" xyz="0 0.001 -0.03595"/>
       <parent link="${side}_index1_link"/>
@@ -210,5 +232,10 @@
     <joint name="${side}_index3_joint" type="revolute">
       <axis xyz="0 1 0"/>
-      <limit effort="1000.0" lower="0.1" upper="-1.5" velocity="0.5"/>
+        <xacro:if value="${side == 'l'}">
+          <limit effort="1000.0" lower="${l_index_joint_lower}" upper="${l_index_joint_upper}" velocity="${l_index_joint_velocity}" />
+        </xacro:if>
+        <xacro:if value="${side == 'r'}">
+          <limit effort="1000.0" lower="${r_index_joint_lower}" upper="${r_index_joint_upper}" velocity="${r_index_joint_velocity}" />
+        </xacro:if>
       <origin rpy="0 0 0" xyz="0 0 -0.024"/>
       <mimic joint="${side}_index_joint" multiplier="1" offset="0"/>
@@ -218,5 +245,10 @@
     <joint name="${side}_middle1_joint" type="revolute">
       <axis xyz="0 1 0"/>
-      <limit effort="1000.0" lower="0.1" upper="-1.5" velocity="0.5"/>
+        <xacro:if value="${side == 'l'}">
+          <limit effort="1000.0" lower="${l_middle_joint_lower}" upper="${l_middle_joint_upper}" velocity="${l_middle_joint_velocity}" />
+        </xacro:if>
+        <xacro:if value="${side == 'r'}">
+          <limit effort="1000.0" lower="${r_middle_joint_lower}" upper="${r_middle_joint_upper}" velocity="${r_middle_joint_velocity}" />
+        </xacro:if>
       <origin rpy="0 0 0" xyz="-0.00175 ${flip * 0.007}  -0.12325"/>
       <mimic joint="${side}_middle_joint" multiplier="1" offset="0"/>
@@ -226,5 +258,10 @@
     <joint name="${side}_middle_joint" type="revolute">
       <axis xyz="0 1 0"/>
-      <limit effort="1000.0" lower="-0.1" upper="1.5" velocity="0.5"/>
+        <xacro:if value="${side == 'l'}">
+          <limit effort="1000.0" lower="${l_middle_joint_lower}" upper="${l_middle_joint_upper}" velocity="${l_middle_joint_velocity}" />
+        </xacro:if>
+        <xacro:if value="${side == 'r'}">
+          <limit effort="1000.0" lower="${r_middle_joint_lower}" upper="${r_middle_joint_upper}" velocity="${r_middle_joint_velocity}" />
+        </xacro:if>
       <origin rpy="0 0 0" xyz="0 0.000 -0.0389"/>
       <parent link="${side}_middle1_link"/>
@@ -233,5 +270,10 @@
     <joint name="${side}_middle3_joint" type="revolute">
       <axis xyz="0 1 0"/>
-      <limit effort="1000.0" lower="-1.57" upper="0.1" velocity="0.5"/>
+        <xacro:if value="${side == 'l'}">
+          <limit effort="1000.0" lower="${l_middle_joint_lower}" upper="${l_middle_joint_upper}" velocity="${l_middle_joint_velocity}" />
+        </xacro:if>
+        <xacro:if value="${side == 'r'}">
+          <limit effort="1000.0" lower="${r_middle_joint_lower}" upper="${r_middle_joint_upper}" velocity="${r_middle_joint_velocity}" />
+        </xacro:if>
       <origin rpy="0 0 0" xyz="0 0.0005 -0.0259"/>
       <mimic joint="${side}_middle_joint" multiplier="1" offset="0"/>
@@ -241,5 +283,10 @@
     <joint name="${side}_ring1_joint" type="revolute">
       <axis xyz="0 0 1"/>
-      <limit effort="1000.0" lower="${flip *-1.57}" upper="0" velocity="0.5"/>
+        <xacro:if value="${side == 'l'}">
+          <limit effort="1000.0" lower="${l_ring_joint_lower}" upper="${l_ring_joint_upper}" velocity="${l_ring_joint_velocity}" />
+        </xacro:if>
+        <xacro:if value="${side == 'r'}">
+          <limit effort="1000.0" lower="${r_ring_joint_lower}" upper="${r_ring_joint_upper}" velocity="${r_ring_joint_velocity}" />
+        </xacro:if>
       <origin rpy="${flip * 0.7} 0 0" xyz="0 ${flip * -0.00705} -0.0794"/>
       <mimic joint="${side}_ring_joint" multiplier="${flip * -0.1}" offset="0"/>
@@ -249,5 +296,10 @@
     <joint name="${side}_ring_joint" type="revolute">
       <axis xyz="0 1 0"/>
-      <limit effort="1000.0" lower="-0.1" upper="1.5" velocity="0.5"/>
+        <xacro:if value="${side == 'l'}">
+          <limit effort="1000.0" lower="${l_ring_joint_lower}" upper="${l_ring_joint_upper}" velocity="${l_ring_joint_velocity}" />
+        </xacro:if>
+        <xacro:if value="${side == 'r'}">
+          <limit effort="1000.0" lower="${r_ring_joint_lower}" upper="${r_ring_joint_upper}" velocity="${r_ring_joint_velocity}" />
+        </xacro:if>
       <origin rpy="${flip * -0.7775} 0 0" xyz="0.00126 ${flip * -0.0351} -0.0166"/>
       <parent link="${side}_ring1_link"/>
@@ -256,5 +308,10 @@
     <joint name="${side}_ring3_joint" type="revolute">
       <axis xyz="0 1 0"/>
-      <limit effort="1000.0" lower="-1.57" upper="0" velocity="0.5"/>
+        <xacro:if value="${side == 'l'}">
+          <limit effort="1000.0" lower="${l_ring_joint_lower}" upper="${l_ring_joint_upper}" velocity="${l_ring_joint_velocity}" />
+        </xacro:if>
+        <xacro:if value="${side == 'r'}">
+          <limit effort="1000.0" lower="${r_ring_joint_lower}" upper="${r_ring_joint_upper}" velocity="${r_ring_joint_velocity}" />
+        </xacro:if>
       <origin rpy="0 0 0" xyz="0 0.0005 -0.0345"/>
       <mimic joint="${side}_ring_joint" multiplier="1" offset="0"/>
@@ -264,5 +321,10 @@
     <joint name="${side}_ring4_joint" type="revolute">
       <axis xyz="0 1 0"/>
-      <limit effort="1000.0" lower="-1.57" upper="0" velocity="0.5"/>
+        <xacro:if value="${side == 'l'}">
+          <limit effort="1000.0" lower="${l_ring_joint_lower}" upper="${l_ring_joint_upper}" velocity="${l_ring_joint_velocity}" />
+        </xacro:if>
+        <xacro:if value="${side == 'r'}">
+          <limit effort="1000.0" lower="${r_ring_joint_lower}" upper="${r_ring_joint_upper}" velocity="${r_ring_joint_velocity}" />
+        </xacro:if>
       <origin rpy="0 0 0" xyz="0 0.0004 -0.0229"/>
       <mimic joint="${side}_ring_joint" multiplier="1" offset="0"/>
@@ -272,5 +334,10 @@
     <joint name="${side}_pinky1_joint" type="revolute">
       <axis xyz="0 0 1"/>
-      <limit effort="1000.0" lower="${flip *-1.57}" upper="0" velocity="0.5"/>
+        <xacro:if value="${side == 'l'}">
+          <limit effort="1000.0" lower="${l_pinky_joint_lower}" upper="${l_pinky_joint_upper}" velocity="${l_pinky_joint_velocity}" />
+        </xacro:if>
+        <xacro:if value="${side == 'r'}">
+          <limit effort="1000.0" lower="${r_pinky_joint_lower}" upper="${r_pinky_joint_upper}" velocity="${r_pinky_joint_velocity}" />
+        </xacro:if>
       <origin rpy="${flip * 0.7} 0 0" xyz="0 ${flip * -0.0270} -0.0555"/>
       <mimic joint="${side}_pinky_joint" multiplier="${flip * -0.1}" offset="0"/>
@@ -280,5 +347,10 @@
     <joint name="${side}_pinky_joint" type="revolute">
       <axis xyz="0 1 0"/>
-      <limit effort="1000.0" lower="-0.1" upper="1.5" velocity="0.5"/>
+        <xacro:if value="${side == 'l'}">
+          <limit effort="1000.0" lower="${l_pinky_joint_lower}" upper="${l_pinky_joint_upper}" velocity="${l_pinky_joint_velocity}" />
+        </xacro:if>
+        <xacro:if value="${side == 'r'}">
+          <limit effort="1000.0" lower="${r_pinky_joint_lower}" upper="${r_pinky_joint_upper}" velocity="${r_pinky_joint_velocity}" />
+        </xacro:if>
       <origin rpy="${flip * -0.93} 0 0" xyz="0 ${flip * -0.046} -0.0228"/>
       <parent link="${side}_pinky1_link"/>
@@ -287,5 +359,10 @@
     <joint name="${side}_pinky3_joint" type="revolute">
       <axis xyz="0 1 0"/>
-      <limit effort="1000.0" lower="-1.57" upper="0" velocity="0.5"/>
+        <xacro:if value="${side == 'l'}">
+          <limit effort="1000.0" lower="${l_pinky_joint_lower}" upper="${l_pinky_joint_upper}" velocity="${l_pinky_joint_velocity}" />
+        </xacro:if>
+        <xacro:if value="${side == 'r'}">
+          <limit effort="1000.0" lower="${r_pinky_joint_lower}" upper="${r_pinky_joint_upper}" velocity="${r_pinky_joint_velocity}" />
+        </xacro:if>
       <origin rpy="0 0 0" xyz="0 0.0005 -0.031"/>
       <mimic joint="${side}_pinky_joint" multiplier="1" offset="0"/>
@@ -295,5 +372,10 @@
     <joint name="${side}_pinky4_joint" type="revolute">
       <axis xyz="0 1 0"/>
-      <limit effort="1000.0" lower="-1.57" upper="0" velocity="0.5"/>
+        <xacro:if value="${side == 'l'}">
+          <limit effort="1000.0" lower="${l_pinky_joint_lower}" upper="${l_pinky_joint_upper}" velocity="${l_pinky_joint_velocity}" />
+        </xacro:if>
+        <xacro:if value="${side == 'r'}">
+          <limit effort="1000.0" lower="${r_pinky_joint_lower}" upper="${r_pinky_joint_upper}" velocity="${r_pinky_joint_velocity}" />
+        </xacro:if>
       <origin rpy="0 0 0" xyz="0 0.0004 -0.0208"/>
       <mimic joint="${side}_pinky_joint" multiplier="1" offset="0"/>

File: inmoov_description/urdf/asmHead.urdf.xacro (robot description, xacro)
@@ -2,4 +2,5 @@
 <robot name="inmoov" xmlns:xacro="http://ros.org/wiki/xacro">
 <xacro:include filename="$(find inmoov_description)/urdf/materials.urdf.xacro" />
+<xacro:include filename="$(find inmoov_description)/urdf/config.urdf.xacro" />
 <xacro:macro name="head" params="covers">
   <link name="head_base_link">
@@ -59,5 +60,5 @@
   <joint name="head_pan_joint" type="revolute">
    <axis xyz="0 0 1"/>
-   <limit effort="1000.0" lower="-1.57" upper="1.57" velocity="0.5"/>
+   <limit effort="1000.0" lower="${head_pan_joint_lower}" upper="${head_pan_joint_upper}" velocity="${head_pan_joint_velocity}" />
    <origin rpy="0 0 0" xyz="0 0 0.0245"/>
    <parent link="head_base_link"/>
@@ -66,5 +67,5 @@
   <joint name="jaw_joint" type="revolute">
    <axis xyz="0 1 0"/>
-   <limit effort="1000.0" lower="0" upper="0.15" velocity="0.5"/>
+   <limit effort="1000.0" lower="${jaw_joint_lower}" upper="${jaw_joint_upper}" velocity="${jaw_joint_velocity}" />
    <origin rpy="0 0.09 0" xyz="0.0375 0.0005 0.0437"/>
    <parent link="head_link"/>
