Commit message: urdf joint vars now defined from config.yaml
not the most elegant solution, but joint limits and velocity are set through config.yaml

File: inmoov_description/urdf/asmTorso.urdf.xacro (robot description, xacro)
@@ -2,4 +2,5 @@
 <robot name="inmoov" xmlns:xacro="http://ros.org/wiki/xacro">
 <xacro:include filename="$(find inmoov_description)/urdf/materials.urdf.xacro" />
+<xacro:include filename="$(find inmoov_description)/urdf/config.urdf.xacro" />
 <xacro:macro name="torso" params="covers">
   <link name="mid_stomach_link">
@@ -75,8 +76,8 @@
     </visual>
   </link>
-  <joint name="waist_rotate_joint" type="revolute">
+  <joint name="waist_pan_joint" type="revolute">
    <axis xyz="0 0 1"/>
-<limit effort="1000.0" lower="-1.57" upper="1.57" velocity="0.5"/>
-      <origin rpy="0 0 0" xyz="0 0 1.152"/>
+   <limit effort="1000.0" lower="${waist_pan_joint_lower}" upper="${waist_pan_joint_upper}" velocity="${waist_pan_joint_velocity}" />
+   <origin rpy="0 0 0" xyz="0 0 1.152"/>
     <parent link="mid_stomach_link"/>
     <child link="top_stomach_link"/>
@@ -87,8 +88,8 @@
     <child link="disk_link"/>
   </joint>
-  <joint name="waist_lean_joint" type="revolute">
+  <joint name="waist_roll_joint" type="revolute">
    <axis xyz="1 0 0"/>
-<limit effort="1000.0" lower="-0.30" upper="0.30" velocity="0.5"/>
-<origin rpy="0 0 0" xyz="0 0 0.11"/>
+   <limit effort="1000.0" lower="${waist_roll_joint_lower}" upper="${waist_roll_joint_upper}" velocity="${waist_roll_joint_velocity}" />
+   <origin rpy="0 0 0" xyz="0 0 0.11"/>
     <parent link="top_stomach_link"/>
     <child link="torso_link"/>

File: inmoov_description/urdf/config.urdf.xacro (robot description, xacro)
@@ -1,4 +1,97 @@
 <?xml version="1.0"?>
 <robot xmlns:xacro="http://ros.org/wiki/xacro">
-  <xacro:include filename="$(find inmoov_bringup)/config/config.xacro" />
+  <xacro:property name="filename" value="$(find inmoov_bringup)/config/config.yaml"/>
+  <xacro:property name="c" value="${load_yaml(filename)}"/>
+  <!--xacro:property name="pi" value="3.1415926539"/-->
+  <xacro:if value="${c['bringup']['angles'] == 'degrees'}">
+    <xacro:property name="r" value="${pi/180.0}"/>
+  </xacro:if>
+  <xacro:if value="${c['bringup']['angles'] == 'radians'}">
+    <xacro:property name="r" value="1"/>
+  </xacro:if>
+  <xacro:property name="r" value="${pi/180.0}"/>
+  <xacro:property name="r_middle_joint_lower"            value="${r*c['joints']['r_middle_joint']['minGoal']}" />
+  <xacro:property name="r_middle_joint_upper"            value="${r*c['joints']['r_middle_joint']['maxGoal']}" />
+  <xacro:property name="r_middle_joint_velocity"         value="${r*c['joints']['r_middle_joint']['maxSpeed']}" />
+  <xacro:property name="r_shoulder_lift_joint_lower"     value="${r*c['joints']['r_shoulder_lift_joint']['minGoal']}" />
+  <xacro:property name="r_shoulder_lift_joint_upper"     value="${r*c['joints']['r_shoulder_lift_joint']['maxGoal']}" />
+  <xacro:property name="r_shoulder_lift_joint_velocity"  value="${r*c['joints']['r_shoulder_lift_joint']['maxSpeed']}" />
+  <xacro:property name="l_ring_joint_lower"              value="${r*c['joints']['l_ring_joint']['minGoal']}" />
+  <xacro:property name="l_ring_joint_upper"              value="${r*c['joints']['l_ring_joint']['maxGoal']}" />
+  <xacro:property name="l_ring_joint_velocity"           value="${r*c['joints']['l_ring_joint']['maxSpeed']}" />
+  <xacro:property name="l_index_joint_lower"             value="${r*c['joints']['l_index_joint']['minGoal']}" />
+  <xacro:property name="l_index_joint_upper"             value="${r*c['joints']['l_index_joint']['maxGoal']}" />
+  <xacro:property name="l_index_joint_velocity"          value="${r*c['joints']['l_index_joint']['maxSpeed']}" />
+  <xacro:property name="head_roll_joint_lower"           value="${r*c['joints']['head_roll_joint']['minGoal']}" />
+  <xacro:property name="head_roll_joint_upper"           value="${r*c['joints']['head_roll_joint']['maxGoal']}" />
+  <xacro:property name="head_roll_joint_velocity"        value="${r*c['joints']['head_roll_joint']['maxSpeed']}" />
+  <xacro:property name="waist_roll_joint_lower"          value="${r*c['joints']['waist_roll_joint']['minGoal']}" />
+  <xacro:property name="waist_roll_joint_upper"          value="${r*c['joints']['waist_roll_joint']['maxGoal']}" />
+  <xacro:property name="waist_roll_joint_velocity"       value="${r*c['joints']['waist_roll_joint']['maxSpeed']}" />
+  <xacro:property name="r_wrist_roll_joint_lower"        value="${r*c['joints']['r_wrist_roll_joint']['minGoal']}" />
+  <xacro:property name="r_wrist_roll_joint_upper"        value="${r*c['joints']['r_wrist_roll_joint']['maxGoal']}" />
+  <xacro:property name="r_wrist_roll_joint_velocity"     value="${r*c['joints']['r_wrist_roll_joint']['maxSpeed']}" />
+  <xacro:property name="l_middle_joint_lower"            value="${r*c['joints']['l_middle_joint']['minGoal']}" />
+  <xacro:property name="l_middle_joint_upper"            value="${r*c['joints']['l_middle_joint']['maxGoal']}" />
+  <xacro:property name="l_middle_joint_velocity"         value="${r*c['joints']['l_middle_joint']['maxSpeed']}" />
+  <xacro:property name="l_thumb_joint_lower"             value="${r*c['joints']['l_thumb_joint']['minGoal']}" />
+  <xacro:property name="l_thumb_joint_upper"             value="${r*c['joints']['l_thumb_joint']['maxGoal']}" />
+  <xacro:property name="l_thumb_joint_velocity"          value="${r*c['joints']['l_thumb_joint']['maxSpeed']}" />
+  <xacro:property name="l_elbow_flex_joint_lower"        value="${r*c['joints']['l_elbow_flex_joint']['minGoal']}" />
+  <xacro:property name="l_elbow_flex_joint_upper"        value="${r*c['joints']['l_elbow_flex_joint']['maxGoal']}" />
+  <xacro:property name="l_elbow_flex_joint_velocity"     value="${r*c['joints']['l_elbow_flex_joint']['maxSpeed']}" />
+  <xacro:property name="jaw_joint_lower"                 value="${r*c['joints']['jaw_joint']['minGoal']}" />
+  <xacro:property name="jaw_joint_upper"                 value="${r*c['joints']['jaw_joint']['maxGoal']}" />
+  <xacro:property name="jaw_joint_velocity"              value="${r*c['joints']['jaw_joint']['maxSpeed']}" />
+  <xacro:property name="l_wrist_roll_joint_lower"        value="${r*c['joints']['l_wrist_roll_joint']['minGoal']}" />
+  <xacro:property name="l_wrist_roll_joint_upper"        value="${r*c['joints']['l_wrist_roll_joint']['maxGoal']}" />
+  <xacro:property name="l_wrist_roll_joint_velocity"     value="${r*c['joints']['l_wrist_roll_joint']['maxSpeed']}" />
+  <xacro:property name="r_elbow_flex_joint_lower"        value="${r*c['joints']['r_elbow_flex_joint']['minGoal']}" />
+  <xacro:property name="r_elbow_flex_joint_upper"        value="${r*c['joints']['r_elbow_flex_joint']['maxGoal']}" />
+  <xacro:property name="r_elbow_flex_joint_velocity"     value="${r*c['joints']['r_elbow_flex_joint']['maxSpeed']}" />
+  <xacro:property name="eyes_pan_joint_lower"            value="${r*c['joints']['eyes_pan_joint']['minGoal']}" />
+  <xacro:property name="eyes_pan_joint_upper"            value="${r*c['joints']['eyes_pan_joint']['maxGoal']}" />
+  <xacro:property name="eyes_pan_joint_velocity"         value="${r*c['joints']['eyes_pan_joint']['maxSpeed']}" />
+  <xacro:property name="r_ring_joint_lower"              value="${r*c['joints']['r_ring_joint']['minGoal']}" />
+  <xacro:property name="r_ring_joint_upper"              value="${r*c['joints']['r_ring_joint']['maxGoal']}" />
+  <xacro:property name="r_ring_joint_velocity"           value="${r*c['joints']['r_ring_joint']['maxSpeed']}" />
+  <xacro:property name="l_shoulder_lift_joint_lower"     value="${r*c['joints']['l_shoulder_lift_joint']['minGoal']}" />
+  <xacro:property name="l_shoulder_lift_joint_upper"     value="${r*c['joints']['l_shoulder_lift_joint']['maxGoal']}" />
+  <xacro:property name="l_shoulder_lift_joint_velocity"  value="${r*c['joints']['l_shoulder_lift_joint']['maxSpeed']}" />
+  <xacro:property name="eyes_tilt_joint_lower"           value="${r*c['joints']['eyes_tilt_joint']['minGoal']}" />
+  <xacro:property name="eyes_tilt_joint_upper"           value="${r*c['joints']['eyes_tilt_joint']['maxGoal']}" />
+  <xacro:property name="eyes_tilt_joint_velocity"        value="${r*c['joints']['eyes_tilt_joint']['maxSpeed']}" />
+  <xacro:property name="r_index_joint_lower"             value="${r*c['joints']['r_index_joint']['minGoal']}" />
+  <xacro:property name="r_index_joint_upper"             value="${r*c['joints']['r_index_joint']['maxGoal']}" />
+  <xacro:property name="r_index_joint_velocity"          value="${r*c['joints']['r_index_joint']['maxSpeed']}" />
+  <xacro:property name="l_pinky_joint_lower"             value="${r*c['joints']['l_pinky_joint']['minGoal']}" />
+  <xacro:property name="l_pinky_joint_upper"             value="${r*c['joints']['l_pinky_joint']['maxGoal']}" />
+  <xacro:property name="l_pinky_joint_velocity"          value="${r*c['joints']['l_pinky_joint']['maxSpeed']}" />
+  <xacro:property name="head_pan_joint_lower"            value="${r*c['joints']['head_pan_joint']['minGoal']}" />
+  <xacro:property name="head_pan_joint_upper"            value="${r*c['joints']['head_pan_joint']['maxGoal']}" />
+  <xacro:property name="head_pan_joint_velocity"         value="${r*c['joints']['head_pan_joint']['maxSpeed']}" />
+  <xacro:property name="r_pinky_joint_lower"             value="${r*c['joints']['r_pinky_joint']['minGoal']}" />
+  <xacro:property name="r_pinky_joint_upper"             value="${r*c['joints']['r_pinky_joint']['maxGoal']}" />
+  <xacro:property name="r_pinky_joint_velocity"          value="${r*c['joints']['r_pinky_joint']['maxSpeed']}" />
+  <xacro:property name="l_shoulder_out_joint_lower"      value="${r*c['joints']['l_shoulder_out_joint']['minGoal']}" />
+  <xacro:property name="l_shoulder_out_joint_upper"      value="${r*c['joints']['l_shoulder_out_joint']['maxGoal']}" />
+  <xacro:property name="l_shoulder_out_joint_velocity"   value="${r*c['joints']['l_shoulder_out_joint']['maxSpeed']}" />
+  <xacro:property name="waist_pan_joint_lower"           value="${r*c['joints']['waist_pan_joint']['minGoal']}" />
+  <xacro:property name="waist_pan_joint_upper"           value="${r*c['joints']['waist_pan_joint']['maxGoal']}" />
+  <xacro:property name="waist_pan_joint_velocity"        value="${r*c['joints']['waist_pan_joint']['maxSpeed']}" />
+  <xacro:property name="r_thumb_joint_lower"             value="${r*c['joints']['r_thumb_joint']['minGoal']}" />
+  <xacro:property name="r_thumb_joint_upper"             value="${r*c['joints']['r_thumb_joint']['maxGoal']}" />
+  <xacro:property name="r_thumb_joint_velocity"          value="${r*c['joints']['r_thumb_joint']['maxSpeed']}" />
+  <xacro:property name="r_upper_arm_roll_joint_lower"    value="${r*c['joints']['r_upper_arm_roll_joint']['minGoal']}" />
+  <xacro:property name="r_upper_arm_roll_joint_upper"    value="${r*c['joints']['r_upper_arm_roll_joint']['maxGoal']}" />
+  <xacro:property name="r_upper_arm_roll_joint_velocity" value="${r*c['joints']['r_upper_arm_roll_joint']['maxSpeed']}" />
+  <xacro:property name="l_upper_arm_roll_joint_lower"    value="${r*c['joints']['l_upper_arm_roll_joint']['minGoal']}" />
+  <xacro:property name="l_upper_arm_roll_joint_upper"    value="${r*c['joints']['l_upper_arm_roll_joint']['maxGoal']}" />
+  <xacro:property name="l_upper_arm_roll_joint_velocity" value="${r*c['joints']['l_upper_arm_roll_joint']['maxSpeed']}" />
+  <xacro:property name="head_tilt_joint_lower"           value="${r*c['joints']['head_tilt_joint']['minGoal']}" />
+  <xacro:property name="head_tilt_joint_upper"           value="${r*c['joints']['head_tilt_joint']['maxGoal']}" />
+  <xacro:property name="head_tilt_joint_velocity"        value="${r*c['joints']['head_tilt_joint']['maxSpeed']}" />
+  <xacro:property name="r_shoulder_out_joint_lower"      value="${r*c['joints']['r_shoulder_out_joint']['minGoal']}" />
+  <xacro:property name="r_shoulder_out_joint_upper"      value="${r*c['joints']['r_shoulder_out_joint']['maxGoal']}" />
+  <xacro:property name="r_shoulder_out_joint_velocity"   value="${r*c['joints']['r_shoulder_out_joint']['maxSpeed']}" />
 </robot>

Commit message: gazebo model improvements
linked to world, added inmoov.gazebo for color definitions

File: inmoov_description/robots/inmoov.urdf.xacro (robot description, xacro)
@@ -4,4 +4,5 @@
 <xacro:include filename="$(find inmoov_description)/urdf/config.inertial.urdf.xacro" />
 <xacro:include filename="$(find inmoov_description)/urdf/materials.urdf.xacro" />
+<xacro:include filename="$(find inmoov_description)/urdf/inmoov.gazebo" />
   <xacro:include filename="$(find inmoov_description)/urdf/materials.urdf.xacro" />
   <xacro:include filename="$(find inmoov_description)/urdf/asmBase.urdf.xacro" />
@@ -12,4 +13,9 @@
   <xacro:include filename="$(find inmoov_description)/urdf/asmArm.urdf.xacro" />
   <xacro:include filename="$(find inmoov_description)/urdf/asmHand.urdf.xacro" />
+  <link name="world"/>
+  <joint name="fixed" type="fixed">
+    <parent link="world"/>
+    <child link="base_link"/>
+  </joint>
   <link name="base_link">
     <visual>
