Commit message: urdf fixes
fixes to xacro fles for kinetic compatibility

File: inmoov_description/urdf/asmArm.urdf.xacro (robot description, xacro)
@@ -26,5 +26,5 @@
         <mesh filename="package://inmoov_description/meshes/bicep.stl" scale="0.001 0.001 0.001"/>
       </geometry>
-      <origin rpy="0 ${(flip * 1.57) + 1.57)} 0" xyz="0 0 0"/>
+      <origin rpy="0 ${(flip * 1.57) + 1.57} 0" xyz="0 0 0"/>
       <xacro:frame_color/>
     </visual>
@@ -35,5 +35,5 @@
         <mesh filename="package://inmoov_description/meshes/bicepcover.stl" scale="0.001 0.001 0.001"/>
       </geometry>
-      <origin rpy="0 ${(flip * 1.57) + 1.57)} 0" xyz="0 0 0"/>
+      <origin rpy="0 ${(flip * 1.57) + 1.57} 0" xyz="0 0 0"/>
       <xacro:cover_color/>
     </visual>
@@ -58,5 +58,5 @@
     <axis xyz="0 0 1"/>
     <limit effort="1000.0" lower="-1.57" upper="1.57" velocity="0.5"/>
-    <origin rpy="0 ${(flip * 1.57) + 1.57)} 0" xyz="${flip * 0.066} 0 -0.060"/>
+    <origin rpy="0 ${(flip * 1.57) + 1.57} 0" xyz="${flip * 0.066} 0 -0.060"/>
     <parent link="${side}_shoulder"/>
     <child link="${side}_bicep"/>
@@ -65,5 +65,5 @@
     <axis xyz="1 0 0"/>
     <limit effort="1000.0" lower="0.4" upper="1.57" velocity="0.5"/>
-    <origin rpy="0 ${(flip * 1.57) + 1.57)} 0" xyz="0 -0.0278 ${flip * 0.2235}"/>
+    <origin rpy="0 ${(flip * 1.57) + 1.57} 0" xyz="0 -0.0278 ${flip * 0.2235}"/>
     <parent link="${side}_bicep"/>
     <child link="${side}_forearm"/>

File: inmoov_description/urdf/materials.urdf.xacro (robot description, xacro)
@@ -1,5 +1,4 @@
 <?xml version="1.0"?>
 <robot xmlns:xacro="http://ros.org/wiki/xacro">
-<xacro:property name="pi" value="3.1415926535897931" />
 <xacro:macro name="decimalrgba" params="r g b a">
       <color rgba="${r/255} ${g/255} ${b/255} ${a/255}"/>
