Commit message: URDF fixes
remove old duplicate stls, flip left thumb cover stl, edits to xacro files

File: inmoov_description/urdf/asmHand.urdf.xacro (robot description, xacro)
@@ -476,5 +476,5 @@
     </joint>
     <joint name="${side}_cover_thumb_joint" type="fixed">
-      <origin rpy="0.05 0 0" xyz="0.01 ${flip * 0.02125} 0.0047"/>
+      <origin rpy="${flip * 0.05} 0 0" xyz="0.01 ${flip * 0.02125} 0.0047"/>
       <parent link="${side}_thumb1_link"/>
       <child link="${side}_cover_thumb_link"/>
