Commit message: URDF Edits for iai_kinect2 rviz
kinect2_ir_optical_frame and kinect2_rgb_optical_frame must have that exact name for the depth cloud mapping to work.

File: inmoov_description/urdf/asmTorso.urdf.xacro (robot description, xacro)
@@ -52,5 +52,5 @@
     <xacro:kinectone_inertial/>
   </link>
-  <link name="kinect2_ir_optical_frame_link">
+  <link name="kinect2_ir_optical_frame">
     <visual>
       <geometry>
@@ -62,5 +62,5 @@
     <xacro:kinectone_inertial/>
   </link>
-  <link name="kinect2_rgb_optical_frame_link">
+  <link name="kinect2_rgb_optical_frame">
     <visual>
       <geometry>
@@ -114,10 +114,10 @@
 <origin rpy="-1.57 0 -1.57" xyz="0 0 0.066"/>
     <parent link="torso_link"/>
-    <child link="kinect2_ir_optical_frame_link"/>
+    <child link="kinect2_ir_optical_frame"/>
   </joint>
   <joint name="kinect2_rgb_optical_joint" type="fixed">
 <origin rpy="-1.57 0 -1.57" xyz="0 0 0.066"/>
     <parent link="torso_link"/>
-    <child link="kinect2_rgb_optical_frame_link"/>
+    <child link="kinect2_rgb_optical_frame"/>
   </joint>
 </xacro:macro>
